File: CON_MOTOR.sch (KiCad schematic (older format))
At the start: 1 part, among them P3 CONN_01X03

Commit message: long forgotten commit of something I did half a year ago -.-
Parts:
- P3: footprint Terminal_Blocks:TerminalBlock_Pheonix_MPT-2.54mm_3pol -> Connector_PinHeader_2.54mm:PinHeader_1x03_P2.54mm_Horizontal; symbol CONN_01X03 -> bldc-controller-rescue:CONN_01X03
Connections:
- net A: now also P3.3 (P3); no longer P3.1 (P1)
- net C: now also P3.1 (P1); no longer P3.3 (P3)
Changed lines of the file:
@@
-EESchema Schematic File Version 2
-LIBS:bldc-controller-rescue
-LIBS:power
-LIBS:device
-LIBS:transistors
-LIBS:conn
-LIBS:linear
-LIBS:regul
-LIBS:74xx
-LIBS:cmos4000
-LIBS:adc-dac
-LIBS:memory
-LIBS:xilinx
-LIBS:microcontrollers
-LIBS:dsp
-LIBS:microchip
-LIBS:analog_switches
-LIBS:motorola
-LIBS:texas
-LIBS:intel
-LIBS:audio
-LIBS:interface
-LIBS:digital-audio
-LIBS:philips
-LIBS:display
-LIBS:cypress
-LIBS:siliconi
-LIBS:opto
-LIBS:atmel
-LIBS:contrib
-LIBS:valves
-LIBS:Power_Management
-LIBS:st-microelectronics
-LIBS:stm32
-LIBS:w_analog
-LIBS:mpu6000
+EESchema Schematic File Version 4
 LIBS:bldc-controller-cache
-EELAYER 25 0
+EELAYER 29 0
 EELAYER END
 $Descr A4 11693 8268
@@
 	1100 700  1000 700
 $Comp
-L CONN_01X03 P3
+L bldc-controller-rescue:CONN_01X03 P3
 U 1 1 5809465E
 P 1300 800
 F 0 "P3" H 1300 1000 50  0000 C CNN
 F 1 "CONN_01X03" V 1400 800 50  0000 C CNN
-F 2 "Terminal_Blocks:TerminalBlock_Pheonix_MPT-2.54mm_3pol" H 1300 800 50  0001 C CNN
+F 2 "Connector_PinHeader_2.54mm:PinHeader_1x03_P2.54mm_Horizontal" H 1300 800 50  0001 C CNN
 F 3 "" H 1300 800 50  0000 C CNN
 	1    1300 800
-	1    0    0    1
+	1    0    0    -1
 $EndComp
 $EndSCHEMATC
