File: Power.sch (KiCad schematic (older format))
At the start: 5 parts, among them P7 CON_PWR_BRD, U7 LD1117S33TR

Commit message: blubb
Parts:
- P7: footprint Connectors_Molex:Molex_KK_6410-04 -> Connectors_Molex:Molex_KK-6410-04_04x2.54mm_Straight
Connections:
- net VPP: now reaches D8.2 (A), P7.2 (P2)
- net +5V: no longer names the net of C13.1, D8.1 (K), U7.3 (VI)
Other:
- moved on the sheet: D8
Changed lines of the file:
@@
 EESchema Schematic File Version 2
+LIBS:bldc-controller-rescue
 LIBS:power
 LIBS:device
@@
 LIBS:st-microelectronics
 LIBS:stm32
+LIBS:w_analog
+LIBS:mpu6000
 LIBS:bldc-controller-cache
 EELAYER 25 0
@@
 $Descr A4 11693 8268
 encoding utf-8
-Sheet 6 6
+Sheet 6 13
 Title ""
 Date ""
@@
 F 0 "P7" H 850 6950 50  0000 C CNN
 F 1 "CON_PWR_BRD" V 950 6700 50  0000 C CNN
-F 2 "Connectors_Molex:Molex_KK_6410-04" H 850 6700 50  0001 C CNN
+F 2 "Connectors_Molex:Molex_KK-6410-04_04x2.54mm_Straight" H 850 6700 50  0001 C CNN
 F 3 "" H 850 6700 50  0000 C CNN
 	1    850  6700
 	-1   0    0    1
 $EndComp
-Wire Wire Line
-	1050 6850 1350 6850
-Wire Wire Line
-	1350 6850 1350 7050
-$Comp
-L GND #PWR050
+$Comp
+L GND #PWR027
 U 1 1 577ED085
 P 1350 7050
-F 0 "#PWR050" H 1350 6800 50  0001 C CNN
+F 0 "#PWR027" H 1350 6800 50  0001 C CNN
 F 1 "GND" H 1350 6900 50  0000 C CNN
 F 2 "" H 1350 7050 50  0000 C CNN
@@
 L D D8
 U 1 1 577ED1D3
-P 1500 6750
-F 0 "D8" H 1500 6850 50  0000 C CNN
-F 1 "D" H 1500 6650 50  0000 C CNN
-F 2 "Diodes_SMD:SOD-323" H 1500 6750 50  0001 C CNN
-F 3 "" H 1500 6750 50  0000 C CNN
-	1    1500 6750
+P 1600 6750
+F 0 "D8" H 1600 6850 50  0000 C CNN
+F 1 "D" H 1600 6650 50  0000 C CNN
+F 2 "Diodes_SMD:SOD-323" H 1600 6750 50  0001 C CNN
+F 3 "" H 1600 6750 50  0000 C CNN
+	1    1600 6750
 	-1   0    0    1
 $EndComp
-Wire Wire Line
-	1050 6750 1350 6750
 $Comp
 L C C13
@@
 $EndComp
 $Comp
-L GND #PWR051
+L GND #PWR028
 U 1 1 577ED346
 P 1800 7150
-F 0 "#PWR051" H 1800 6900 50  0001 C CNN
+F 0 "#PWR028" H 1800 6900 50  0001 C CNN
 F 1 "GND" H 1800 7000 50  0000 C CNN
 F 2 "" H 1800 7150 50  0000 C CNN
@@
 $EndComp
 $Comp
-L GND #PWR052
+L GND #PWR029
 U 1 1 577ED360
 P 2800 7150
-F 0 "#PWR052" H 2800 6900 50  0001 C CNN
+F 0 "#PWR029" H 2800 6900 50  0001 C CNN
 F 1 "GND" H 2800 7000 50  0000 C CNN
 F 2 "" H 2800 7150 50  0000 C CNN
@@
 $EndComp
 $Comp
-L GND #PWR053
+L GND #PWR030
 U 1 1 577ED37A
 P 2300 7150
-F 0 "#PWR053" H 2300 6900 50  0001 C CNN
+F 0 "#PWR030" H 2300 6900 50  0001 C CNN
 F 1 "GND" H 2300 7000 50  0000 C CNN
 F 2 "" H 2300 7150 50  0000 C CNN
@@
 	1    0    0    -1
 $EndComp
-Wire Wire Line
-	2300 7050 2300 7150
-Wire Wire Line
-	1800 7100 1800 7150
-Wire Wire Line
-	2800 7100 2800 7150
-Wire Wire Line
-	2700 6750 2950 6750
-Wire Wire Line
-	2800 6750 2800 6800
-Wire Wire Line
-	1650 6750 1900 6750
-Wire Wire Line
-	1800 6550 1800 6800
-Connection ~ 1800 6750
-$Comp
-L +5V #PWR054
-U 1 1 577ED523
-P 1800 6550
-F 0 "#PWR054" H 1800 6400 50  0001 C CNN
-F 1 "+5V" H 1800 6690 50  0000 C CNN
-F 2 "" H 1800 6550 50  0000 C CNN
-F 3 "" H 1800 6550 50  0000 C CNN
-	1    1800 6550
-	1    0    0    -1
-$EndComp
-$Comp
-L VCC #PWR055
+$Comp
+L VCC #PWR032
 U 1 1 577ED553
 P 2950 6550
-F 0 "#PWR055" H 2950 6400 50  0001 C CNN
+F 0 "#PWR032" H 2950 6400 50  0001 C CNN
 F 1 "VCC" H 2950 6700 50  0000 C CNN
 F 2 "" H 2950 6550 50  0000 C CNN
@@
 	1    0    0    -1
 $EndComp
-Wire Wire Line
-	2950 6750 2950 6550
-Connection ~ 2800 6750
 Text HLabel 1300 6350 1    60   Input ~ 0
 RX_PWR_BOARD
 Text HLabel 1150 6350 1    60   Input ~ 0
 TX_PWR_BOARD
-Wire Wire Line
-	1150 6350 1150 6550
-Wire Wire Line
-	1150 6550 1050 6550
-Wire Wire Line
-	1300 6350 1300 6650
-Wire Wire Line
-	1300 6650 1050 6650
 $Comp
 L LD1117S33TR U7
@@
 	1    0    0    -1
 $EndComp
+$Comp
+L PWR_FLAG #FLG034
+U 1 1 57B4ECE8
+P 1150 7050
+F 0 "#FLG034" H 1150 7145 50  0001 C CNN
+F 1 "PWR_FLAG" H 1150 7230 50  0000 C CNN
+F 2 "" H 1150 7050 50  0000 C CNN
+F 3 "" H 1150 7050 50  0000 C CNN
+	1    1150 7050
+	-1   0    0    1
+$EndComp
+$Comp
+L VPP #PWR?
+U 1 1 57B36023
+P 1400 6400
+F 0 "#PWR?" H 1400 6250 50  0001 C CNN
+F 1 "VPP" H 1400 6550 50  0000 C CNN
+F 2 "" H 1400 6400 50  0000 C CNN
+F 3 "" H 1400 6400 50  0000 C CNN
+	1    1400 6400
+	1    0    0    -1
+$EndComp
+Wire Wire Line
+	1050 6850 1350 6850
+Wire Wire Line
+	1350 6850 1350 7050
+Wire Wire Line
+	1050 6750 1450 6750
+Wire Wire Line
+	2300 7050 2300 7150
+Wire Wire Line
+	1800 7100 1800 7150
+Wire Wire Line
+	2800 7100 2800 7150
+Wire Wire Line
+	2700 6750 2950 6750
+Wire Wire Line
+	1750 6750 1900 6750
+Connection ~ 1800 6750
+Wire Wire Line
+	2950 6750 2950 6550
+Connection ~ 2800 6750
+Wire Wire Line
+	1150 6350 1150 6550
+Wire Wire Line
+	1150 6550 1050 6550
+Wire Wire Line
+	1300 6350 1300 6650
+Wire Wire Line
+	1300 6650 1050 6650
+Wire Wire Line
+	1150 7050 1150 7000
+Wire Wire Line
+	1150 7000 1350 7000
+Connection ~ 1350 7000
+Wire Wire Line
+	2800 6800 2800 6750
+Wire Wire Line
+	1800 6800 1800 6750
+Wire Wire Line
+	1400 6400 1400 6750
+Connection ~ 1400 6750
 $EndSCHEMATC

Commit message: routed
Connections:
- net VPP: no longer D8.2 (A)
- net +5V: now reaches C13.1, D8.1 (K), U7.3 (VI)
- net RX_PWR_BOARD: no longer names the net of P7.3 (P3)
- net RX_PWR_BOARD: now also D8.2 (A)
- net TX_PWR_BOARD renamed RX_TX_PWR_BOARD
Changed lines of the file:
@@
 $Descr A4 11693 8268
 encoding utf-8
-Sheet 6 13
+Sheet 6 12
 Title ""
 Date ""
@@
 $EndComp
 $Comp
-L GND #PWR027
+L GND #PWR026
 U 1 1 577ED085
 P 1350 7050
-F 0 "#PWR027" H 1350 6800 50  0001 C CNN
+F 0 "#PWR026" H 1350 6800 50  0001 C CNN
 F 1 "GND" H 1350 6900 50  0000 C CNN
 F 2 "" H 1350 7050 50  0000 C CNN
@@
 $EndComp
 $Comp
-L GND #PWR028
+L GND #PWR027
 U 1 1 577ED346
 P 1800 7150
-F 0 "#PWR028" H 1800 6900 50  0001 C CNN
+F 0 "#PWR027" H 1800 6900 50  0001 C CNN
 F 1 "GND" H 1800 7000 50  0000 C CNN
 F 2 "" H 1800 7150 50  0000 C CNN
@@
 $EndComp
 $Comp
-L GND #PWR029
+L GND #PWR028
 U 1 1 577ED360
 P 2800 7150
-F 0 "#PWR029" H 2800 6900 50  0001 C CNN
+F 0 "#PWR028" H 2800 6900 50  0001 C CNN
 F 1 "GND" H 2800 7000 50  0000 C CNN
 F 2 "" H 2800 7150 50  0000 C CNN
@@
 $EndComp
 $Comp
-L GND #PWR030
+L GND #PWR029
 U 1 1 577ED37A
 P 2300 7150
-F 0 "#PWR030" H 2300 6900 50  0001 C CNN
+F 0 "#PWR029" H 2300 6900 50  0001 C CNN
 F 1 "GND" H 2300 7000 50  0000 C CNN
 F 2 "" H 2300 7150 50  0000 C CNN
@@
 $EndComp
 $Comp
-L VCC #PWR032
+L VCC #PWR030
 U 1 1 577ED553
 P 2950 6550
-F 0 "#PWR032" H 2950 6400 50  0001 C CNN
+F 0 "#PWR030" H 2950 6400 50  0001 C CNN
 F 1 "VCC" H 2950 6700 50  0000 C CNN
 F 2 "" H 2950 6550 50  0000 C CNN
@@
 	1    0    0    -1
 $EndComp
-Text HLabel 1300 6350 1    60   Input ~ 0
-RX_PWR_BOARD
-Text HLabel 1150 6350 1    60   Input ~ 0
-TX_PWR_BOARD
+Text HLabel 1100 6350 1    60   Input ~ 0
+RX_TX_PWR_BOARD
 $Comp
 L LD1117S33TR U7
@@
 $EndComp
 $Comp
-L PWR_FLAG #FLG034
+L PWR_FLAG #FLG031
 U 1 1 57B4ECE8
 P 1150 7050
-F 0 "#FLG034" H 1150 7145 50  0001 C CNN
+F 0 "#FLG031" H 1150 7145 50  0001 C CNN
 F 1 "PWR_FLAG" H 1150 7230 50  0000 C CNN
 F 2 "" H 1150 7050 50  0000 C CNN
@@
 $EndComp
 $Comp
-L VPP #PWR?
+L VPP #PWR032
 U 1 1 57B36023
-P 1400 6400
-F 0 "#PWR?" H 1400 6250 50  0001 C CNN
-F 1 "VPP" H 1400 6550 50  0000 C CNN
-F 2 "" H 1400 6400 50  0000 C CNN
-F 3 "" H 1400 6400 50  0000 C CNN
-	1    1400 6400
+P 1200 6400
+F 0 "#PWR032" H 1200 6250 50  0001 C CNN
+F 1 "VPP" H 1200 6550 50  0000 C CNN
+F 2 "" H 1200 6400 50  0000 C CNN
+F 3 "" H 1200 6400 50  0000 C CNN
+	1    1200 6400
 	1    0    0    -1
 $EndComp
@@
 	1350 6850 1350 7050
 Wire Wire Line
-	1050 6750 1450 6750
+	1200 6750 1050 6750
 Wire Wire Line
 	2300 7050 2300 7150
@@
 Connection ~ 2800 6750
 Wire Wire Line
-	1150 6350 1150 6550
-Wire Wire Line
-	1150 6550 1050 6550
-Wire Wire Line
-	1300 6350 1300 6650
-Wire Wire Line
-	1300 6650 1050 6650
+	1100 6350 1100 6550
+Wire Wire Line
+	1100 6550 1050 6550
+Wire Wire Line
+	1050 6650 1450 6650
 Wire Wire Line
 	1150 7050 1150 7000
@@
 	2800 6800 2800 6750
 Wire Wire Line
-	1800 6800 1800 6750
-Wire Wire Line
-	1400 6400 1400 6750
-Connection ~ 1400 6750
+	1200 6400 1200 6750
+$Comp
+L +5V #PWR033
+U 1 1 57B42FF7
+P 1800 6200
+F 0 "#PWR033" H 1800 6050 50  0001 C CNN
+F 1 "+5V" H 1800 6340 50  0000 C CNN
+F 2 "" H 1800 6200 50  0000 C CNN
+F 3 "" H 1800 6200 50  0000 C CNN
+	1    1800 6200
+	1    0    0    -1
+$EndComp
+$Comp
+L PWR_FLAG #FLG034
+U 1 1 57B47DFF
+P 1950 5450
+F 0 "#FLG034" H 1950 5545 50  0001 C CNN
+F 1 "PWR_FLAG" H 1950 5630 50  0000 C CNN
+F 2 "" H 1950 5450 50  0000 C CNN
+F 3 "" H 1950 5450 50  0000 C CNN
+	1    1950 5450
+	0    1    1    0
+$EndComp
+$Comp
+L PWR_FLAG #FLG035
+U 1 1 57B47E75
+P 1950 5850
+F 0 "#FLG035" H 1950 5945 50  0001 C CNN
+F 1 "PWR_FLAG" H 1950 6030 50  0000 C CNN
+F 2 "" H 1950 5850 50  0000 C CNN
+F 3 "" H 1950 5850 50  0000 C CNN
+	1    1950 5850
+	0    1    1    0
+$EndComp
+Wire Wire Line
+	1450 5850 1450 6750
+$Comp
+L PWR_FLAG #FLG036
+U 1 1 57B49678
+P 1950 6250
+F 0 "#FLG036" H 1950 6345 50  0001 C CNN
+F 1 "PWR_FLAG" H 1950 6430 50  0000 C CNN
+F 2 "" H 1950 6250 50  0000 C CNN
+F 3 "" H 1950 6250 50  0000 C CNN
+	1    1950 6250
+	0    1    1    0
+$EndComp
+Wire Wire Line
+	1800 6200 1800 6800
+Wire Wire Line
+	1950 6250 1800 6250
+Connection ~ 1800 6250
+Wire Wire Line
+	1450 5850 1950 5850
+Connection ~ 1450 6650
+Wire Wire Line
+	1200 6450 1350 6450
+Wire Wire Line
+	1350 6450 1350 5450
+Wire Wire Line
+	1350 5450 1950 5450
+Connection ~ 1200 6450
 $EndSCHEMATC

Commit message: blubb
Connections:
- net +5VA: now reaches D8.2 (A), P7.3 (P3)
Other:
- note added: ""unsafe 5V""
Changed lines of the file:
@@
 $EndComp
 $Comp
-L GND #PWR026
+L GND #PWR027
 U 1 1 577ED085
 P 1350 7050
-F 0 "#PWR026" H 1350 6800 50  0001 C CNN
+F 0 "#PWR027" H 1350 6800 50  0001 C CNN
 F 1 "GND" H 1350 6900 50  0000 C CNN
 F 2 "" H 1350 7050 50  0000 C CNN
@@
 $EndComp
 $Comp
-L GND #PWR027
+L GND #PWR028
 U 1 1 577ED346
 P 1800 7150
-F 0 "#PWR027" H 1800 6900 50  0001 C CNN
+F 0 "#PWR028" H 1800 6900 50  0001 C CNN
 F 1 "GND" H 1800 7000 50  0000 C CNN
 F 2 "" H 1800 7150 50  0000 C CNN
@@
 $EndComp
 $Comp
-L GND #PWR028
+L GND #PWR029
 U 1 1 577ED360
 P 2800 7150
-F 0 "#PWR028" H 2800 6900 50  0001 C CNN
+F 0 "#PWR029" H 2800 6900 50  0001 C CNN
 F 1 "GND" H 2800 7000 50  0000 C CNN
 F 2 "" H 2800 7150 50  0000 C CNN
@@
 $EndComp
 $Comp
-L GND #PWR029
+L GND #PWR030
 U 1 1 577ED37A
 P 2300 7150
-F 0 "#PWR029" H 2300 6900 50  0001 C CNN
+F 0 "#PWR030" H 2300 6900 50  0001 C CNN
 F 1 "GND" H 2300 7000 50  0000 C CNN
 F 2 "" H 2300 7150 50  0000 C CNN
@@
 $EndComp
 $Comp
-L VCC #PWR030
+L VCC #PWR031
 U 1 1 577ED553
 P 2950 6550
-F 0 "#PWR030" H 2950 6400 50  0001 C CNN
+F 0 "#PWR031" H 2950 6400 50  0001 C CNN
 F 1 "VCC" H 2950 6700 50  0000 C CNN
 F 2 "" H 2950 6550 50  0000 C CNN
@@
 $EndComp
 $Comp
-L PWR_FLAG #FLG031
+L PWR_FLAG #FLG032
 U 1 1 57B4ECE8
 P 1150 7050
-F 0 "#FLG031" H 1150 7145 50  0001 C CNN
+F 0 "#FLG032" H 1150 7145 50  0001 C CNN
 F 1 "PWR_FLAG" H 1150 7230 50  0000 C CNN
 F 2 "" H 1150 7050 50  0000 C CNN
@@
 $EndComp
 $Comp
-L VPP #PWR032
+L VPP #PWR033
 U 1 1 57B36023
 P 1200 6400
-F 0 "#PWR032" H 1200 6250 50  0001 C CNN
+F 0 "#PWR033" H 1200 6250 50  0001 C CNN
 F 1 "VPP" H 1200 6550 50  0000 C CNN
 F 2 "" H 1200 6400 50  0000 C CNN
@@
 	1200 6400 1200 6750
 $Comp
-L +5V #PWR033
+L +5V #PWR034
 U 1 1 57B42FF7
 P 1800 6200
-F 0 "#PWR033" H 1800 6050 50  0001 C CNN
+F 0 "#PWR034" H 1800 6050 50  0001 C CNN
 F 1 "+5V" H 1800 6340 50  0000 C CNN
 F 2 "" H 1800 6200 50  0000 C CNN
@@
 $EndComp
 $Comp
-L PWR_FLAG #FLG034
+L PWR_FLAG #FLG035
 U 1 1 57B47DFF
 P 1950 5450
-F 0 "#FLG034" H 1950 5545 50  0001 C CNN
+F 0 "#FLG035" H 1950 5545 50  0001 C CNN
 F 1 "PWR_FLAG" H 1950 5630 50  0000 C CNN
 F 2 "" H 1950 5450 50  0000 C CNN
@@
 $EndComp
 $Comp
-L PWR_FLAG #FLG035
+L PWR_FLAG #FLG036
 U 1 1 57B47E75
 P 1950 5850
-F 0 "#FLG035" H 1950 5945 50  0001 C CNN
+F 0 "#FLG036" H 1950 5945 50  0001 C CNN
 F 1 "PWR_FLAG" H 1950 6030 50  0000 C CNN
 F 2 "" H 1950 5850 50  0000 C CNN
@@
 	1450 5850 1450 6750
 $Comp
-L PWR_FLAG #FLG036
+L PWR_FLAG #FLG037
 U 1 1 57B49678
 P 1950 6250
-F 0 "#FLG036" H 1950 6345 50  0001 C CNN
+F 0 "#FLG037" H 1950 6345 50  0001 C CNN
 F 1 "PWR_FLAG" H 1950 6430 50  0000 C CNN
 F 2 "" H 1950 6250 50  0000 C CNN
@@
 	1350 5450 1950 5450
 Connection ~ 1200 6450
+$Comp
+L +5VA #PWR?
+U 1 1 57B577AF
+P 1800 5750
+F 0 "#PWR?" H 1800 5600 50  0001 C CNN
+F 1 "+5VA" H 1800 5890 50  0000 C CNN
+F 2 "" H 1800 5750 50  0000 C CNN
+F 3 "" H 1800 5750 50  0000 C CNN
+	1    1800 5750
+	1    0    0    -1
+$EndComp
+Wire Wire Line
+	1800 5750 1800 5850
+Connection ~ 1800 5850
+Text Notes 1500 5800 0    60   ~ 0
+"unsafe 5V"
 $EndSCHEMATC

Commit message: bestellversion
Connections:
- net +5VA: now also P7.2 (P2); no longer P7.3 (P3)
- net VPP: now also P7.3 (P3); no longer P7.2 (P2)
Changed lines of the file:
@@
 	1350 6850 1350 7050
-Wire Wire Line
-	1200 6750 1050 6750
 Wire Wire Line
 	2300 7050 2300 7150
@@
 	1100 6550 1050 6550
 Wire Wire Line
-	1050 6650 1450 6650
-Wire Wire Line
 	1150 7050 1150 7000
 Wire Wire Line
@@
 	2800 6800 2800 6750
 Wire Wire Line
-	1200 6400 1200 6750
+	1200 6400 1200 6650
 $Comp
 L +5V #PWR034
@@
 Wire Wire Line
 	1450 5850 1950 5850
-Connection ~ 1450 6650
 Wire Wire Line
 	1200 6450 1350 6450
@@
 Text Notes 1500 5800 0    60   ~ 0
 "unsafe 5V"
+Wire Wire Line
+	1200 6650 1050 6650
+Wire Wire Line
+	1450 6750 1050 6750
 $EndSCHEMATC

Commit message: updated some stuff and added some more docu
Parts:
- removed D8: D, Diodes_SMD:SOD-323, symbol D
- added D5: D_Small, Diodes_SMD:SOD-323, symbol D_Small
Connections:
- net +5V: now also D5.1 (K)
- net +5VA: now also D5.2 (A)
Changed lines of the file:
@@
-$EndComp
-$Comp
-L D D8
-U 1 1 577ED1D3
-P 1600 6750
-F 0 "D8" H 1600 6850 50  0000 C CNN
-F 1 "D" H 1600 6650 50  0000 C CNN
-F 2 "Diodes_SMD:SOD-323" H 1600 6750 50  0001 C CNN
-F 3 "" H 1600 6750 50  0000 C CNN
-	1    1600 6750
-	-1   0    0    1
 $EndComp
 $Comp
@@
 	2700 6750 2950 6750
 Wire Wire Line
-	1750 6750 1900 6750
+	1700 6750 1900 6750
 Connection ~ 1800 6750
 Wire Wire Line
@@
 	1200 6650 1050 6650
 Wire Wire Line
-	1450 6750 1050 6750
+	1050 6750 1500 6750
+$Comp
+L D_Small D5
+U 1 1 57BAD647
+P 1600 6750
+F 0 "D5" H 1550 6830 50  0000 L CNN
+F 1 "D_Small" H 1450 6670 50  0000 L CNN
+F 2 "Diodes_SMD:SOD-323" V 1600 6750 50  0001 C CNN
+F 3 "" V 1600 6750 50  0000 C CNN
+	1    1600 6750
+	-1   0    0    1
+$EndComp
+Connection ~ 1450 6750
 $EndSCHEMATC

Commit message: routed... at least for now
Parts:
- P7: footprint Connectors_Molex:Molex_KK-6410-04_04x2.54mm_Straight -> Terminal_Blocks:TerminalBlock_Pheonix_MPT-2.54mm_4pol
Changed lines of the file:
@@
 $Descr A4 11693 8268
 encoding utf-8
-Sheet 6 12
+Sheet 5 12
 Title ""
 Date ""
@@
 F 0 "P7" H 850 6950 50  0000 C CNN
 F 1 "CON_PWR_BRD" V 950 6700 50  0000 C CNN
-F 2 "Connectors_Molex:Molex_KK-6410-04_04x2.54mm_Straight" H 850 6700 50  0001 C CNN
+F 2 "Terminal_Blocks:TerminalBlock_Pheonix_MPT-2.54mm_4pol" H 850 6700 50  0001 C CNN
 F 3 "" H 850 6700 50  0000 C CNN
 	1    850  6700
@@
 $EndComp
 $Comp
-L GND #PWR027
+L GND #PWR021
 U 1 1 577ED085
 P 1350 7050
-F 0 "#PWR027" H 1350 6800 50  0001 C CNN
+F 0 "#PWR021" H 1350 6800 50  0001 C CNN
 F 1 "GND" H 1350 6900 50  0000 C CNN
 F 2 "" H 1350 7050 50  0000 C CNN
@@
 $EndComp
 $Comp
-L GND #PWR028
+L GND #PWR022
 U 1 1 577ED346
 P 1800 7150
-F 0 "#PWR028" H 1800 6900 50  0001 C CNN
+F 0 "#PWR022" H 1800 6900 50  0001 C CNN
 F 1 "GND" H 1800 7000 50  0000 C CNN
 F 2 "" H 1800 7150 50  0000 C CNN
@@
 $EndComp
 $Comp
-L GND #PWR029
+L GND #PWR023
 U 1 1 577ED360
 P 2800 7150
-F 0 "#PWR029" H 2800 6900 50  0001 C CNN
+F 0 "#PWR023" H 2800 6900 50  0001 C CNN
 F 1 "GND" H 2800 7000 50  0000 C CNN
 F 2 "" H 2800 7150 50  0000 C CNN
@@
 $EndComp
 $Comp
-L GND #PWR030
+L GND #PWR024
 U 1 1 577ED37A
 P 2300 7150
-F 0 "#PWR030" H 2300 6900 50  0001 C CNN
+F 0 "#PWR024" H 2300 6900 50  0001 C CNN
 F 1 "GND" H 2300 7000 50  0000 C CNN
 F 2 "" H 2300 7150 50  0000 C CNN
@@
 $EndComp
 $Comp
-L VCC #PWR031
+L VCC #PWR025
 U 1 1 577ED553
 P 2950 6550
-F 0 "#PWR031" H 2950 6400 50  0001 C CNN
+F 0 "#PWR025" H 2950 6400 50  0001 C CNN
 F 1 "VCC" H 2950 6700 50  0000 C CNN
 F 2 "" H 2950 6550 50  0000 C CNN
@@
 $EndComp
 $Comp
-L PWR_FLAG #FLG032
+L PWR_FLAG #FLG026
 U 1 1 57B4ECE8
 P 1150 7050
-F 0 "#FLG032" H 1150 7145 50  0001 C CNN
+F 0 "#FLG026" H 1150 7145 50  0001 C CNN
 F 1 "PWR_FLAG" H 1150 7230 50  0000 C CNN
 F 2 "" H 1150 7050 50  0000 C CNN
@@
 $EndComp
 $Comp
-L VPP #PWR033
+L VPP #PWR027
 U 1 1 57B36023
 P 1200 6400
-F 0 "#PWR033" H 1200 6250 50  0001 C CNN
+F 0 "#PWR027" H 1200 6250 50  0001 C CNN
 F 1 "VPP" H 1200 6550 50  0000 C CNN
 F 2 "" H 1200 6400 50  0000 C CNN
@@
 	1200 6400 1200 6650
 $Comp
-L +5V #PWR034
+L +5V #PWR028
 U 1 1 57B42FF7
 P 1800 6200
-F 0 "#PWR034" H 1800 6050 50  0001 C CNN
+F 0 "#PWR028" H 1800 6050 50  0001 C CNN
 F 1 "+5V" H 1800 6340 50  0000 C CNN
 F 2 "" H 1800 6200 50  0000 C CNN
@@
 $EndComp
 $Comp
-L PWR_FLAG #FLG035
+L PWR_FLAG #FLG029
 U 1 1 57B47DFF
 P 1950 5450
-F 0 "#FLG035" H 1950 5545 50  0001 C CNN
+F 0 "#FLG029" H 1950 5545 50  0001 C CNN
 F 1 "PWR_FLAG" H 1950 5630 50  0000 C CNN
 F 2 "" H 1950 5450 50  0000 C CNN
@@
 $EndComp
 $Comp
-L PWR_FLAG #FLG036
+L PWR_FLAG #FLG030
 U 1 1 57B47E75
 P 1950 5850
-F 0 "#FLG036" H 1950 5945 50  0001 C CNN
+F 0 "#FLG030" H 1950 5945 50  0001 C CNN
 F 1 "PWR_FLAG" H 1950 6030 50  0000 C CNN
 F 2 "" H 1950 5850 50  0000 C CNN
@@
 	1450 5850 1450 6750
 $Comp
-L PWR_FLAG #FLG037
+L PWR_FLAG #FLG031
 U 1 1 57B49678
 P 1950 6250
-F 0 "#FLG037" H 1950 6345 50  0001 C CNN
+F 0 "#FLG031" H 1950 6345 50  0001 C CNN
 F 1 "PWR_FLAG" H 1950 6430 50  0000 C CNN
 F 2 "" H 1950 6250 50  0000 C CNN
@@
 Connection ~ 1200 6450
 $Comp
-L +5VA #PWR038
+L +5VA #PWR032
 U 1 1 57B577AF
 P 1800 5750
-F 0 "#PWR038" H 1800 5600 50  0001 C CNN
+F 0 "#PWR032" H 1800 5600 50  0001 C CNN
 F 1 "+5VA" H 1800 5890 50  0000 C CNN
 F 2 "" H 1800 5750 50  0000 C CNN
