File: driver.sch (KiCad schematic (older format))
At the start: 17 parts, among them IC1 L6205PD

Commit message: blubb
Parts:
- removed C?: 4.7uF, symbol CP1_Small
- added C22: 4.7uF, Capacitors_SMD:C_0805, symbol C_Small
- C1, C2: footprint (none) -> Capacitors_SMD:C_0603
- C18, C19, C20, C21: renamed from C?; footprint (none) -> Capacitors_SMD:C_0603
- D1, D2: footprint (none) -> Diodes_SMD:SOD-323
- IC1: footprint st-microelectronics-POWERSO-20 -> BLDC:SOIC-20
- R1: footprint (none) -> Resistors_SMD:R_0603
- R10, R11, R8, R9: renamed from R?; footprint (none) -> Resistors_SMD:R_1206
- R6, R7: renamed from R?; footprint (none) -> Resistors_SMD:R_0603
Connections:
- net GND: now also C22.2
- net VPP: now also C22.1
Changed lines of the file:
@@
 EESchema Schematic File Version 2
+LIBS:bldc-controller-rescue
 LIBS:power
 LIBS:device
@@
 LIBS:st-microelectronics
 LIBS:stm32
+LIBS:w_analog
+LIBS:mpu6000
 LIBS:bldc-controller-cache
 EELAYER 25 0
@@
 $Descr A4 11693 8268
 encoding utf-8
-Sheet 2 6
+Sheet 2 13
 Title ""
 Date ""
@@
 F 0 "IC1" V 1900 2500 50  0000 L BNN
 F 1 "L6205PD" V 2465 1750 50  0000 L BNN
-F 2 "st-microelectronics-POWERSO-20" H 2500 2100 50  0001 C CNN
+F 2 "BLDC:SOIC-20" H 2500 2100 50  0001 C CNN
 F 3 "" H 2500 1950 60  0000 C CNN
 	1    2500 1950
@@
 F 0 "C2" H 1660 1720 50  0000 L CNN
 F 1 "10nF" H 1660 1570 50  0000 L CNN
-F 2 "" H 1650 1650 50  0000 C CNN
+F 2 "Capacitors_SMD:C_0603" H 1650 1650 50  0001 C CNN
 F 3 "" H 1650 1650 50  0000 C CNN
 	1    1650 1650
@@
 F 0 "D1" H 950 1630 50  0000 L CNN
 F 1 "D_Small" H 850 1470 50  0000 L CNN
-F 2 "" V 1000 1550 50  0000 C CNN
+F 2 "Diodes_SMD:SOD-323" V 1000 1550 50  0001 C CNN
 F 3 "" V 1000 1550 50  0000 C CNN
 	1    1000 1550
@@
 F 0 "R1" H 1430 1670 50  0000 L CNN
 F 1 "100" H 1430 1610 50  0000 L CNN
-F 2 "" H 1400 1650 50  0000 C CNN
+F 2 "Resistors_SMD:R_0603" H 1400 1650 50  0001 C CNN
 F 3 "" H 1400 1650 50  0000 C CNN
 	1    1400 1650
@@
 	1750 1650 1800 1650
 $Comp
-L VPP #PWR1
+L VPP #PWR011
 U 1 1 578D3DEA
 P 1200 1050
-F 0 "#PWR1" H 1200 900 50  0001 C CNN
+F 0 "#PWR011" H 1200 900 50  0001 C CNN
 F 1 "VPP" H 1200 1200 50  0000 C CNN
 F 2 "" H 1200 1050 50  0000 C CNN
@@
 F 0 "D2" H 1150 1630 50  0000 L CNN
 F 1 "D_Small" H 1050 1470 50  0000 L CNN
-F 2 "" V 1200 1550 50  0000 C CNN
+F 2 "Diodes_SMD:SOD-323" V 1200 1550 50  0001 C CNN
 F 3 "" V 1200 1550 50  0000 C CNN
 	1    1200 1550
@@
 F 0 "C1" H 1210 1320 50  0000 L CNN
 F 1 "220nF" H 1210 1170 50  0000 L CNN
-F 2 "" H 1200 1250 50  0000 C CNN
+F 2 "Capacitors_SMD:C_0603" H 1200 1250 50  0001 C CNN
 F 3 "" H 1200 1250 50  0000 C CNN
 	1    1200 1250
@@
 EN_A
 $Comp
-L VPP #PWR?
+L VPP #PWR012
 U 1 1 578D4588
 P 3350 1150
-F 0 "#PWR?" H 3350 1000 50  0001 C CNN
+F 0 "#PWR012" H 3350 1000 50  0001 C CNN
 F 1 "VPP" H 3350 1300 50  0000 C CNN
 F 2 "" H 3350 1150 50  0000 C CNN
@@
 	3200 2350 3550 2350
 $Comp
-L GND #PWR?
+L GND #PWR013
 U 1 1 578D486E
 P 2450 2750
-F 0 "#PWR?" H 2450 2500 50  0001 C CNN
+F 0 "#PWR013" H 2450 2500 50  0001 C CNN
 F 1 "GND" H 2450 2600 50  0000 C CNN
 F 2 "" H 2450 2750 50  0000 C CNN
@@
 $EndComp
 $Comp
-L C_Small C?
+L C_Small C18
 U 1 1 578D4A26
 P 1550 2650
-F 0 "C?" H 1560 2720 50  0000 L CNN
+F 0 "C18" H 1560 2720 50  0000 L CNN
 F 1 "2nF" H 1560 2570 50  0000 L CNN
-F 2 "" H 1550 2650 50  0000 C CNN
+F 2 "Capacitors_SMD:C_0603" H 1550 2650 50  0001 C CNN
 F 3 "" H 1550 2650 50  0000 C CNN
 	1    1550 2650
@@
 $EndComp
 $Comp
-L R_Small R?
+L R_Small R7
 U 1 1 578D4A59
 P 1300 2450
-F 0 "R?" H 1330 2470 50  0000 L CNN
+F 0 "R7" H 1330 2470 50  0000 L CNN
 F 1 "10k" H 1330 2410 50  0000 L CNN
-F 2 "" H 1300 2450 50  0000 C CNN
+F 2 "Resistors_SMD:R_0603" H 1300 2450 50  0001 C CNN
 F 3 "" H 1300 2450 50  0000 C CNN
 	1    1300 2450
@@
 	1150 2450 1200 2450
 $Comp
-L GND #PWR?
+L GND #PWR014
 U 1 1 578D4B75
 P 1550 2800
-F 0 "#PWR?" H 1550 2550 50  0001 C CNN
+F 0 "#PWR014" H 1550 2550 50  0001 C CNN
 F 1 "GND" H 1550 2650 50  0000 C CNN
 F 2 "" H 1550 2800 50  0000 C CNN
@@
 	1550 2800 1550 2750
 $Comp
-L R_Small R?
+L R_Small R6
 U 1 1 578D4CDE
 P 1300 2050
-F 0 "R?" H 1330 2070 50  0000 L CNN
+F 0 "R6" H 1330 2070 50  0000 L CNN
 F 1 "10k" H 1330 2010 50  0000 L CNN
-F 2 "" H 1300 2050 50  0000 C CNN
+F 2 "Resistors_SMD:R_0603" H 1300 2050 50  0001 C CNN
 F 3 "" H 1300 2050 50  0000 C CNN
 	1    1300 2050
@@
 $EndComp
 $Comp
-L C_Small C?
+L C_Small C19
 U 1 1 578D4D15
 P 1750 2650
-F 0 "C?" H 1760 2720 50  0000 L CNN
+F 0 "C19" H 1760 2720 50  0000 L CNN
 F 1 "2nF" H 1760 2570 50  0000 L CNN
-F 2 "" H 1750 2650 50  0000 C CNN
+F 2 "Capacitors_SMD:C_0603" H 1750 2650 50  0001 C CNN
 F 3 "" H 1750 2650 50  0000 C CNN
 	1    1750 2650
@@
 	1200 2050 1150 2050
 $Comp
-L GND #PWR?
+L GND #PWR015
 U 1 1 578D4EB3
 P 1750 2800
-F 0 "#PWR?" H 1750 2550 50  0001 C CNN
+F 0 "#PWR015" H 1750 2550 50  0001 C CNN
 F 1 "GND" H 1750 2650 50  0000 C CNN
 F 2 "" H 1750 2800 50  0000 C CNN
@@
 	1750 2800 1750 2750
 $Comp
-L C_Small C?
+L C_Small C20
 U 1 1 578D502E
 P 2400 950
-F 0 "C?" H 2410 1020 50  0000 L CNN
+F 0 "C20" H 2410 1020 50  0000 L CNN
 F 1 "100nF" H 2410 870 50  0000 L CNN
-F 2 "" H 2400 950 50  0000 C CNN
+F 2 "Capacitors_SMD:C_0603" H 2400 950 50  0001 C CNN
 F 3 "" H 2400 950 50  0000 C CNN
 	1    2400 950
@@
 $EndComp
 $Comp
-L C_Small C?
+L C_Small C21
 U 1 1 578D5083
 P 2600 950
-F 0 "C?" H 2610 1020 50  0000 L CNN
+F 0 "C21" H 2610 1020 50  0000 L CNN
 F 1 "100nF" H 2610 870 50  0000 L CNN
-F 2 "" H 2600 950 50  0000 C CNN
+F 2 "Capacitors_SMD:C_0603" H 2600 950 50  0001 C CNN
 F 3 "" H 2600 950 50  0000 C CNN
 	1    2600 950
@@
 $EndComp
 $Comp
-L GND #PWR?
+L GND #PWR016
 U 1 1 578D512F
 P 2600 1150
-F 0 "#PWR?" H 2600 900 50  0001 C CNN
+F 0 "#PWR016" H 2600 900 50  0001 C CNN
 F 1 "GND" H 2600 1000 50  0000 C CNN
 F 2 "" H 2600 1150 50  0000 C CNN
@@
 $EndComp
 $Comp
-L VPP #PWR?
+L VPP #PWR017
 U 1 1 578D524A
 P 2600 750
-F 0 "#PWR?" H 2600 600 50  0001 C CNN
+F 0 "#PWR017" H 2600 600 50  0001 C CNN
 F 1 "VPP" H 2600 900 50  0000 C CNN
 F 2 "" H 2600 750 50  0000 C CNN
@@
 $EndComp
 $Comp
-L R_Small R?
+L R_Small R8
 U 1 1 578D546A
 P 3300 2800
-F 0 "R?" H 3330 2820 50  0000 L CNN
+F 0 "R8" H 3330 2820 50  0000 L CNN
 F 1 ".1" H 3330 2760 50  0000 L CNN
-F 2 "" H 3300 2800 50  0000 C CNN
+F 2 "Resistors_SMD:R_1206" H 3300 2800 50  0001 C CNN
 F 3 "" H 3300 2800 50  0000 C CNN
 	1    3300 2800
@@
 $EndComp
 $Comp
-L R_Small R?
+L R_Small R9
 U 1 1 578D54B4
 P 3450 2800
-F 0 "R?" H 3480 2820 50  0000 L CNN
+F 0 "R9" H 3480 2820 50  0000 L CNN
 F 1 ".1" H 3480 2760 50  0000 L CNN
-F 2 "" H 3450 2800 50  0000 C CNN
+F 2 "Resistors_SMD:R_1206" H 3450 2800 50  0001 C CNN
 F 3 "" H 3450 2800 50  0000 C CNN
 	1    3450 2800
@@
 $EndComp
 $Comp
-L R_Small R?
+L R_Small R10
 U 1 1 578D556E
 P 3850 2800
-F 0 "R?" H 3880 2820 50  0000 L CNN
+F 0 "R10" H 3880 2820 50  0000 L CNN
 F 1 ".1" H 3880 2760 50  0000 L CNN
-F 2 "" H 3850 2800 50  0000 C CNN
+F 2 "Resistors_SMD:R_1206" H 3850 2800 50  0001 C CNN
 F 3 "" H 3850 2800 50  0000 C CNN
 	1    3850 2800
@@
 $EndComp
 $Comp
-L R_Small R?
+L R_Small R11
 U 1 1 578D55BF
 P 4000 2800
-F 0 "R?" H 4030 2820 50  0000 L CNN
+F 0 "R11" H 4030 2820 50  0000 L CNN
 F 1 ".1" H 4030 2760 50  0000 L CNN
-F 2 "" H 4000 2800 50  0000 C CNN
+F 2 "Resistors_SMD:R_1206" H 4000 2800 50  0001 C CNN
 F 3 "" H 4000 2800 50  0000 C CNN
 	1    4000 2800
@@
 	3450 2950 3450 2900
 $Comp
-L GND #PWR?
+L GND #PWR018
 U 1 1 578D56C4
 P 3300 3000
-F 0 "#PWR?" H 3300 2750 50  0001 C CNN
+F 0 "#PWR018" H 3300 2750 50  0001 C CNN
 F 1 "GND" H 3300 2850 50  0000 C CNN
 F 2 "" H 3300 3000 50  0000 C CNN
@@
 	4000 2950 4000 2900
 $Comp
-L GND #PWR?
+L GND #PWR019
 U 1 1 578D5888
 P 3850 3000
-F 0 "#PWR?" H 3850 2750 50  0001 C CNN
+F 0 "#PWR019" H 3850 2750 50  0001 C CNN
 F 1 "GND" H 3850 2850 50  0000 C CNN
 F 2 "" H 3850 3000 50  0000 C CNN
@@
 	4050 2550 3300 2550
 Connection ~ 3300 2550
-$Comp
-L CP1_Small C?
-U 1 1 578E56DD
+Wire Wire Line
+	2800 800  2800 850
+Wire Wire Line
+	2400 800  2800 800
+Wire Wire Line
+	2400 850  2400 800
+Wire Wire Line
+	2600 750  2600 850
+Connection ~ 2600 800
+Wire Wire Line
+	2400 1050 2400 1100
+Wire Wire Line
+	2400 1100 2800 1100
+Wire Wire Line
+	2800 1100 2800 1050
+Wire Wire Line
+	2600 1050 2600 1150
+Connection ~ 2600 1100
+Wire Wire Line
+	2450 2700 2450 2750
+Wire Wire Line
+	2300 2700 2600 2700
+Wire Wire Line
+	2600 2700 2600 2650
+Wire Wire Line
+	2300 2700 2300 2650
+Connection ~ 2450 2700
+Wire Wire Line
+	2400 2650 2400 2700
+Connection ~ 2400 2700
+Wire Wire Line
+	2500 2650 2500 2700
+Connection ~ 2500 2700
+$Comp
+L C_Small C22
+U 1 1 57ADFC17
 P 2800 950
-F 0 "C?" H 2810 1020 50  0000 L CNN
+F 0 "C22" H 2810 1020 50  0000 L CNN
 F 1 "4.7uF" H 2810 870 50  0000 L CNN
-F 2 "" H 2800 950 50  0000 C CNN
+F 2 "Capacitors_SMD:C_0805" H 2800 950 50  0001 C CNN
 F 3 "" H 2800 950 50  0000 C CNN
 	1    2800 950
 	1    0    0    -1
 $EndComp
-Wire Wire Line
-	2800 800  2800 850
-Wire Wire Line
-	2400 800  2800 800
-Wire Wire Line
-	2400 850  2400 800
-Wire Wire Line
-	2600 750  2600 850
-Connection ~ 2600 800
-Wire Wire Line
-	2400 1050 2400 1100
-Wire Wire Line
-	2400 1100 2800 1100
-Wire Wire Line
-	2800 1100 2800 1050
-Wire Wire Line
-	2600 1050 2600 1150
-Connection ~ 2600 1100
-Wire Wire Line
-	2450 2750 2450 2700
-Wire Wire Line
-	2300 2700 2600 2700
-Wire Wire Line
-	2600 2700 2600 2650
-Wire Wire Line
-	2300 2700 2300 2650
-Connection ~ 2450 2700
-Wire Wire Line
-	2400 2650 2400 2700
-Connection ~ 2400 2700
-Wire Wire Line
-	2500 2650 2500 2700
-Connection ~ 2500 2700
+$Comp
+L PWR_FLAG #FLG020
+U 1 1 57B20A0F
+P 3550 1200
+F 0 "#FLG020" H 3550 1295 50  0001 C CNN
+F 1 "PWR_FLAG" H 3550 1380 50  0000 C CNN
+F 2 "" H 3550 1200 50  0000 C CNN
+F 3 "" H 3550 1200 50  0000 C CNN
+	1    3550 1200
+	1    0    0    -1
+$EndComp
+Wire Wire Line
+	3550 1200 3550 1300
+Wire Wire Line
+	3550 1300 3350 1300
+Connection ~ 3350 1300
 $EndSCHEMATC

Commit message: routed
Changed lines of the file:
@@
 $Descr A4 11693 8268
 encoding utf-8
-Sheet 2 13
+Sheet 2 12
 Title ""
 Date ""
@@
 	1    0    0    -1
 $EndComp
-$Comp
-L PWR_FLAG #FLG020
-U 1 1 57B20A0F
-P 3550 1200
-F 0 "#FLG020" H 3550 1295 50  0001 C CNN
-F 1 "PWR_FLAG" H 3550 1380 50  0000 C CNN
-F 2 "" H 3550 1200 50  0000 C CNN
-F 3 "" H 3550 1200 50  0000 C CNN
-	1    3550 1200
-	1    0    0    -1
-$EndComp
-Wire Wire Line
-	3550 1200 3550 1300
-Wire Wire Line
-	3550 1300 3350 1300
-Connection ~ 3350 1300
 $EndSCHEMATC

Commit message: bestellversion
Parts:
- C18, C19: value 2nF -> 10nF
Changed lines of the file:
@@
 F 1 "L6205PD" V 2465 1750 50  0000 L BNN
 F 2 "BLDC:SOIC-20" H 2500 2100 50  0001 C CNN
-F 3 "" H 2500 1950 60  0000 C CNN
+F 3 "docs/L6205PD.pdf" H 2450 2150 60  0000 C CNN
 	1    2500 1950
 	1    0    0    -1
@@
 P 1550 2650
 F 0 "C18" H 1560 2720 50  0000 L CNN
-F 1 "2nF" H 1560 2570 50  0000 L CNN
+F 1 "10nF" H 1560 2570 50  0000 L CNN
 F 2 "Capacitors_SMD:C_0603" H 1550 2650 50  0001 C CNN
 F 3 "" H 1550 2650 50  0000 C CNN
@@
 P 1750 2650
 F 0 "C19" H 1760 2720 50  0000 L CNN
-F 1 "2nF" H 1760 2570 50  0000 L CNN
+F 1 "10nF" H 1760 2570 50  0000 L CNN
 F 2 "Capacitors_SMD:C_0603" H 1750 2650 50  0001 C CNN
 F 3 "" H 1750 2650 50  0000 C CNN

Commit message: updated stuff
Parts:
- removed C1: 220nF, Capacitors_SMD:C_0603, symbol C_Small
- removed C18, C19, C2: 10nF, Capacitors_SMD:C_0603, symbol C_Small
- removed C22: 4.7uF, Capacitors_SMD:C_0805, symbol C_Small
- removed D1, D2: D_Small, Diodes_SMD:SOD-323, symbol D_Small
- removed IC1: L6205PD, BLDC:SOIC-20, symbol L6205PD
- removed R1: 100, Resistors_SMD:R_0603, symbol R_Small
- removed R10, R11, R9: .1, Resistors_SMD:R_1206, symbol R_Small
- removed R6, R7: 10k, Resistors_SMD:R_0603, symbol R_Small
- added C? (x3): 2.2uF, Capacitors_SMD:C_0603, symbol C_Small
- added C? (x3): 100nF, Capacitors_SMD:C_0603, symbol C_Small
- added C? (x2): 1nF, Capacitors_SMD:C_0603, symbol C_Small
- added C?: 22nF, Capacitors_SMD:C_0603, symbol C_Small
- added Q? (x6): Q_NMOS_DGS, symbol Q_NMOS_DGS
- added R?: 1R, symbol R_Small
- added R? (x6): 10R, symbol R_Small
- added R?: .01, Resistors_SMD:R_1206, symbol R_Small
- added R? (x2): 10kR, symbol R_Small
- added U?: DRV8313, symbol DRV8313
- C20: value 100nF -> 4.7uF
- R8: value .1 -> .01
Connections:
- net GND: now also C?.1, C?.1, C?.2, C?.2, C?.2, R?.2, R?.2, U?.24 (AGND), U?.26 (SP2), U?.28 (SP1), U?.46 (GND), U?.47 (GND), U?.48 (GND), U?.49 (PPAD)
- net VPP: now also U?.25 (PVDD)
- net SENSE_B: no longer names the net of R8.1
- net SENSE_B: now also C?.2, Q?.3 (S), U?.29 (SN1), U?.40 (SL_A)
- new net: Q?.2 (G), R?.1 (x6)
- new net: C?.1, U?.9 (GVDD)
- new net: C?.1, U?.19 (DVDD)
- new net: C?.1, U?.23 (AVDD)
- new net: C?.1, U?.10 (CP1)
- new net: C?.2, U?.11 (CP2)
- new net: C?.2, Q?.3 (S), R?.1, U?.27 (SN2), U?.35 (SL_B)
- new net: R?.1, U?.3 (DTC)
- new net: Q?.3 (S), U?.30 (SL_C)
- new net: R?.2, U?.31 (GL_C)
- new net: R?.2, U?.33 (GH_C)
- new net: C?.2, U?.34 (BST_C)
- new net: R?.2, U?.36 (GL_B)
- new net: R?.2, U?.38 (GH_B)
- new net: C?.2, U?.39 (BST_B)
- new net: R?.2, U?.41 (GL_A)
- new net: R?.2, U?.43 (GH_A)
- new net: C?.2, U?.44 (BST_A)
- new net DRV_CUR_1: U?.21 (SO1)
- new net DRV_CUR_2: U?.22 (SO2)
- new net DRV_DC_CAL: U?.8 (DC_CAL)
- new net DRV_ENABLE: U?.12 (EN_GATE)
- new net DRV_NCS: U?.4 (nSCS)
- new net DRV_REF_V: U?.20 (REF)
- new net DRV_SCLK: U?.7 (SCKL)
- new net DRV_SDI: U?.5 (SDI)
- new net DRV_SDO: U?.6 (SDO)
- new net IN_H_A: U?.13 (INH_A)
- new net IN_H_B: U?.15 (INH_B)
- new net IN_H_C: U?.17 (INH_C)
- new net IN_L_A: U?.14 (INL_A)
- new net IN_L_B: U?.16 (INL_B)
- new net IN_L_C: U?.18 (INL_C)
- new net OUT_A: C?.1, Q?.1 (D), Q?.3 (S), U?.42 (SH_A)
- new net OUT_B: C?.1, Q?.1 (D), Q?.3 (S), U?.37 (SH_B)
- new net OUT_C: C?.1, Q?.1 (D), Q?.3 (S), U?.32 (SH_C)
- new net VCC: R?.1, R?.1, U?.45 (VDD_SPI)
- new net nFAULT: R?.2, U?.2 (nFAULT)
- new net nOCTW: R?.2, U?.1 (nOCTW)
Other:
- moved on the sheet: C20, C21, R8

Commit message: routed... at least for now
Parts:
- removed C20: 4.7uF, Capacitors_SMD:C_0603, symbol C_Small
- added C20: 10uF, Capacitors_ThroughHole:C_Radial_D5_L11_P2, symbol CP1_Small
- Q1, Q2, Q3, Q4, Q5, Q6: renamed from Q?; footprint (none) -> BLDC:SOT1210
- R10, R11, R13, R14, R2, R4, R6, R7, R9: renamed from R?; footprint (none) -> Resistors_SMD:R_0603
- R12: renamed from R?; footprint Resistors_SMD:R_1206 -> Resistors_SMD:R_1210
- R8: footprint Resistors_SMD:R_1206 -> Resistors_SMD:R_1210
- U2: renamed from U?; footprint (none) -> BLDC:SOIC-48
- gave numbers to parts that had none: 9
Connections:
- net GND: now also U2.27 (SN2), C20.2
- net VPP: now also Q1.1 (D), Q3.1 (D), Q5.1 (D), C20.1
- net at C22.2, Q2.3 (S), R8.1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: now also C23.2, Q4.3 (S), Q6.3 (S), R12.1, U2.30 (SL_C), U2.35 (SL_B)
- net DRV_CUR_2: no longer names the net of U2.22 (SO2)
- no-connect marks 0 -> 1
Other:
- moved on the sheet: C22, C23, Q1, Q2, R12, R7, R8, R9
