File: bldc-controller.kicad_pcb (KiCad board)
At the start: 2 copper layers, 56 x 39 mm, 57 parts, among them IC1 L6205PD, P1 CON_LED, P2 CON_LIDAR, P3 CON_MOTOR, P4 USB_OTG, P5 CON_SWD, P6 CON_HALL, P7 CON_PWR_BRD, U1 STM32F405R, U5 MPU6000, U7 LD1117S33TR, Y1 Crystal

Commit message: routed
Parts:
- removed P2: CON_LIDAR, Connectors_Molex:Molex_KK-6410-07_07x2.54mm_Straight
- C1, C21, D1, D2, D8, R2, R3, R5: moved to B.Cu
- moved U7 38.6 mm to (149.5, 100.0), turned to 90 degrees
- moved C14 38.5 mm to (148.5, 100.0), turned to 0 degrees
- moved C13 36.2 mm to (148.5, 98.5), turned to 0 degrees
- moved D8 24.2 mm to (134.4, 98.0)
- moved C1 19.7 mm to (128.5, 92.0), turned to 270 degrees
- moved D2 17.4 mm to (131.5, 91.5), turned to 0 degrees
- moved D3 17.4 mm to (147.5, 88.0), turned to 90 degrees
- moved D1 15.8 mm to (131.5, 93.0), turned to 0 degrees
- moved R2 15.7 mm to (148.5, 82.5)
- moved R3 15.7 mm to (148.5, 84.0)
- moved R1 13.1 mm to (134.5, 92.5), turned to 90 degrees
- moved R5 12.1 mm to (152.5, 87.0)
- moved C17 9.45 mm to (148.5, 78.5), turned to 180 degrees
- moved C2 9.12 mm to (136.0, 92.5), turned to 270 degrees
- moved R4 7.85 mm to (154.0, 87.0), turned to 270 degrees
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Connections:
- P4 pad 6: Net-(P4-Pad6) -> GND
- P7 pad 2: Net-(D8-Pad2) -> VPP
- P7 pad 3: /Power/RX_PWR_BOARD -> Net-(D8-Pad2)
- P7 pad 4: /Power/TX_PWR_BOARD -> /Power/RX_TX_PWR_BOARD
- U1 pad 14: /Power/RX_PWR_BOARD -> /Power/RX_TX_PWR_BOARD
- U1 pad 15: /Power/RX_PWR_BOARD -> /Power/RX_TX_PWR_BOARD
- U1 pad 16: /Power/TX_PWR_BOARD -> (no net)
- U1 pad 17: /Power/TX_PWR_BOARD -> (no net)
- U1 pad 37: /CON_LIDAR/LIDAR_TX -> (no net)
- U1 pad 38: /CON_LIDAR/LIDAR_RX -> (no net)
- U1 pad 39: /CON_LIDAR/LIDAR_MOTOR_EN -> (no net)
- U1 pad 56: /driver/EN_A -> /driver/EN_B
- U1 pad 57: /driver/EN_B -> /driver/EN_A
- U1 pad 58: /driver/IN1_A -> /driver/IN2_B
- U1 pad 59: /driver/IN2_A -> /driver/IN1_B
- U1 pad 61: /driver/IN1_B -> /driver/IN1_A
- U1 pad 62: /driver/IN2_B -> /driver/IN2_A
Routing:
- net +5V: track 0.00 -> 67.4 mm, vias 0 -> 3
- net /Power/RX_TX_PWR_BOARD: track 0.00 -> 41.4 mm, vias 0 -> 3
- net /CUR_SENSE_4/OUT_2: track 1.76 -> 35.8 mm, vias 0 -> 1
- net /CUR_SENSE_4/OUT_1: track 2.32 -> 35.4 mm, vias 0 -> 1
- net /CUR_SENSE_4/OUT_3: track 1.76 -> 34.6 mm, vias 0 -> 1
- net /driver/IN1_B: track 0.00 -> 32.4 mm, vias 0 -> 2
- net /driver/SENSE_B: track 2.22 -> 34.2 mm, vias 2 -> 3
- net /driver/IN2_B: track 0.00 -> 30.7 mm, vias 0 -> 2
- net /CUR_SENSE_4/OUT_4: track 2.32 -> 32.5 mm, vias 0 -> 1
- net GND: track 2.18 -> 28.5 mm, vias 2 -> 19
- net /driver/EN_A: track 0.00 -> 24.8 mm, vias 0 -> 3
- net /SWDIO/SWDCLK: track 0.00 -> 22.9 mm, vias 0 -> 2
- net /driver/EN_B: track 0.00 -> 21.2 mm, vias 0 -> 1
- net /SWDIO/NRST: track 0.00 -> 19.4 mm, vias 0 -> 3
- net /SWDIO/SWDIO: track 0.00 -> 19.2 mm, vias 0 -> 2
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- added copper zone on F.Cu, net VPP
Other:
- board size 56 x 39 mm -> 47 x 39 mm

Commit message: blubb
Parts:
- removed D5, D6, D7, D9: 3V, Diodes_SMD:SOD-323
- moved D8 8.54 mm to (142.9, 97.8), turned to 180 degrees
- moved C15 3.27 mm to (160.0, 93.8), turned to 180 degrees
Connections:
- D8 pad 2: Net-(D8-Pad2) -> +5VA
- P1 pad 1: +5V -> +5VA
- P7 pad 3: Net-(D8-Pad2) -> +5VA
Routing:
- net +5VA: track 0.00 -> 33.2 mm
- net +5V: track 67.4 -> 54.0 mm
- net /Power/RX_TX_PWR_BOARD: track 41.4 -> 37.2 mm, vias 3 -> 1
- net /CUR_SENSE_4/OUT_2: track 35.8 -> 31.8 mm
- net /CUR_SENSE_4/OUT_3: track 34.6 -> 30.7 mm
- net Net-(C15-Pad1): track 1.87 -> 5.76 mm
- net Net-(D8-Pad2): track 2.92 -> 0.00 mm
- net /CUR_SENSE_4/OUT_1: track 35.4 -> 32.8 mm
- net /CUR_SENSE_4/OUT_4: track 32.5 -> 29.9 mm
- net /IMU/nCS: track 15.7 -> 13.5 mm, vias 3 -> 1
- net GND: track 28.5 -> 27.1 mm, vias 19 -> 18
- net /CON_LED/LED_DATA: track 16.4 -> 17.5 mm
- net /IMU/SDO: track 15.9 -> 14.8 mm
- net /IMU/SCK: track 14.7 -> 13.8 mm
- net /IMU/SDI: track 15.1 -> 14.4 mm
Other:
- rule via_min_size: 0.4 -> 0.6

Commit message: fertig?
Parts:
- added P10: MOUNTING, Connect:1pin, F.Cu at (127.0, 69.0)
- added P11: CONN_01X03, Pin_Headers:Pin_Header_Straight_1x03, F.Cu at (167.0, 90.6)
- added P12: CONN_01X03, Pin_Headers:Pin_Header_Straight_1x03, F.Cu at (164.5, 90.6)
- added P2: MOUNTING, Connect:1pin, F.Cu at (168.0, 102.0)
- added P8: MOUNTING, Connect:1pin, F.Cu at (127.0, 102.0)
- added P9: MOUNTING, Connect:1pin, F.Cu at (168.0, 69.0)
- P1: footprint Connectors_Molex:Molex_KK-6410-03_03x2.54mm_Straight -> Pin_Headers:Pin_Header_Straight_1x03
- moved C11 4.49 mm to (158.7, 91.2), turned to 180 degrees
- moved C15 2.22 mm to (157.8, 93.5), turned to 90 degrees
- moved U5 1.77 mm to (158.6, 92.2)
- moved C16 1.66 mm to (159.3, 93.5), turned to 90 degrees
- moved P7 1.50 mm to (141.0, 102.0)
- moved P1 0.14 mm to (161.6, 101.9), turned to 270 degrees
Connections:
- U1 pad 16: (no net) -> /2CON/SIG_2
- U1 pad 17: (no net) -> /2CON/SIG_1
Routing:
- net +5VA: track 33.2 -> 45.4 mm, vias 0 -> 1
- net /2CON/SIG_2: track 0.00 -> 10.6 mm, vias 0 -> 2
- net /2CON/SIG_1: track 0.00 -> 10.3 mm, vias 0 -> 2
- net /IMU/nCS: track 13.5 -> 10.0 mm
- net /IMU/SDI: track 14.4 -> 17.2 mm
- net /IMU/SDO: track 14.8 -> 12.1 mm
- net GND: track 27.1 -> 29.7 mm, vias 18 -> 19
- net /IMU/SCK: track 13.8 -> 15.8 mm
- net /Power/RX_TX_PWR_BOARD: track 37.2 -> 35.7 mm
- net /driver/IN2_A: track 11.0 -> 12.0 mm
- net VCC: track 18.2 -> 19.0 mm

Commit message: bestellversion
Parts:
- added REF**1111111: VIA-0.6, BLDC:VIA-0.6, F.Cu at (132.0, 94.5)
- added REF**11111111111: VIA-0.6, BLDC:VIA-0.6, F.Cu at (134.0, 87.7)
- added REF**11111111112: VIA-0.6, BLDC:VIA-0.6, F.Cu at (134.0, 88.7)
- added REF**11111111113: VIA-0.6, BLDC:VIA-0.6, F.Cu at (134.0, 89.7)
- added REF**11111111114: VIA-0.6, BLDC:VIA-0.6, F.Cu at (134.0, 90.7)
- added REF**11111111121: VIA-0.6, BLDC:VIA-0.6, F.Cu at (135.0, 87.7)
- added REF**11111111122: VIA-0.6, BLDC:VIA-0.6, F.Cu at (135.0, 88.7)
- added REF**11111111123: VIA-0.6, BLDC:VIA-0.6, F.Cu at (135.0, 89.7)
- added REF**11111111124: VIA-0.6, BLDC:VIA-0.6, F.Cu at (135.0, 90.7)
- added REF**11111111131: VIA-0.6, BLDC:VIA-0.6, F.Cu at (136.0, 87.7)
- added REF**11111111132: VIA-0.6, BLDC:VIA-0.6, F.Cu at (136.0, 88.7)
- added REF**11111111133: VIA-0.6, BLDC:VIA-0.6, F.Cu at (136.0, 89.7)
- added REF**11111111134: VIA-0.6, BLDC:VIA-0.6, F.Cu at (136.0, 90.7)
- added REF**11111111141: VIA-0.6, BLDC:VIA-0.6, F.Cu at (137.0, 87.7)
- added REF**11111111142: VIA-0.6, BLDC:VIA-0.6, F.Cu at (137.0, 88.7)
- added REF**11111111143: VIA-0.6, BLDC:VIA-0.6, F.Cu at (137.0, 89.7)
- added REF**11111111144: VIA-0.6, BLDC:VIA-0.6, F.Cu at (137.0, 90.7)
- added REF**1111112: VIA-0.6, BLDC:VIA-0.6, F.Cu at (132.0, 95.5)
- added REF**1111113: VIA-0.6, BLDC:VIA-0.6, F.Cu at (132.0, 96.5)
- added REF**1111121: VIA-0.6, BLDC:VIA-0.6, F.Cu at (133.0, 94.5)
- added REF**1111122: VIA-0.6, BLDC:VIA-0.6, F.Cu at (133.0, 95.5)
- added REF**1111123: VIA-0.6, BLDC:VIA-0.6, F.Cu at (133.0, 96.5)
- added REF**1111131: VIA-0.6, BLDC:VIA-0.6, F.Cu at (134.0, 94.5)
- added REF**1111132: VIA-0.6, BLDC:VIA-0.6, F.Cu at (134.0, 95.5)
- added REF**1111133: VIA-0.6, BLDC:VIA-0.6, F.Cu at (134.0, 96.5)
- added REF**1111141: VIA-0.6, BLDC:VIA-0.6, F.Cu at (135.0, 94.5)
- added REF**1111142: VIA-0.6, BLDC:VIA-0.6, F.Cu at (135.0, 95.5)
- added REF**1111143: VIA-0.6, BLDC:VIA-0.6, F.Cu at (135.0, 96.5)
- added REF**1111151: VIA-0.6, BLDC:VIA-0.6, F.Cu at (136.0, 94.5)
- added REF**1111152: VIA-0.6, BLDC:VIA-0.6, F.Cu at (136.0, 95.5)
- added REF**1111153: VIA-0.6, BLDC:VIA-0.6, F.Cu at (136.0, 96.5)
- added REF**1111161: VIA-0.6, BLDC:VIA-0.6, F.Cu at (137.0, 94.5)
- added REF**1111162: VIA-0.6, BLDC:VIA-0.6, F.Cu at (137.0, 95.5)
- added REF**1111163: VIA-0.6, BLDC:VIA-0.6, F.Cu at (137.0, 96.5)
- added REF**1111171: VIA-0.6, BLDC:VIA-0.6, F.Cu at (138.0, 94.5)
- added REF**1111172: VIA-0.6, BLDC:VIA-0.6, F.Cu at (138.0, 95.5)
- added REF**1111173: VIA-0.6, BLDC:VIA-0.6, F.Cu at (138.0, 96.5)
- added REF**1111181: VIA-0.6, BLDC:VIA-0.6, F.Cu at (139.0, 94.5)
- added REF**1111182: VIA-0.6, BLDC:VIA-0.6, F.Cu at (139.0, 95.5)
- added REF**1111183: VIA-0.6, BLDC:VIA-0.6, F.Cu at (139.0, 96.5)
- C22, C8, C9: moved to B.Cu
- moved C22 2.10 mm to (146.5, 92.9)
- moved C9 2.06 mm to (152.5, 92.2), turned to 90 degrees
- moved C8 1.87 mm to (151.0, 92.2), turned to 90 degrees
Connections:
- P7 pad 2: VPP -> +5VA
- P7 pad 3: +5VA -> VPP
Routing:
- net GND: track 29.7 -> 25.7 mm, vias 19 -> 16
- net +5VA: track 45.4 -> 42.2 mm
- net VPP: track 8.47 -> 9.92 mm, vias 2 -> 3
- net /OSC/OSC_OUT: track 8.49 -> 9.84 mm, vias 0 -> 1
- net /OSC/OSC_IN: track 8.61 -> 9.94 mm, vias 0 -> 1

Commit message: updated some stuff and added some more docu
Changed lines of the file:
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@@
     (links 198)
     (no_connects 0)
-    (area 123.924999 65.924999 171.075001 105.075001)
+    (area 122.989286 63.92412 184.3 111.800001)
     (thickness 1.6)
     (drawings 6)
@@
     (mod_text_size 1 1)
     (mod_text_width 0.15)
-    (pad_size 4.064 4.064)
-    (pad_drill 3)
+    (pad_size 1.25 1.25)
+    (pad_drill 0.85)
     (pad_to_mask_clearance 0.2)
     (aux_axis_origin 0 0)
@@
     (pad 5 smd rect (at 1.2991 -1.56254 270) (size 1.35 0.4) (layers F.Cu F.Paste F.Mask)
       (net 5 GND))
-    (pad 6 thru_hole oval (at -2.5009 -1.56254 270) (size 0.95 1.25) (drill oval 0.55 0.85) (layers *.Cu *.Mask F.SilkS)
-      (net 5 GND))
-    (pad 6 thru_hole oval (at 2.4991 -1.56254 270) (size 0.95 1.25) (drill oval 0.55 0.85) (layers *.Cu *.Mask F.SilkS)
-      (net 5 GND))
-    (pad 6 thru_hole oval (at -3.5009 1.13746 270) (size 1.55 1) (drill oval 1.15 0.5) (layers *.Cu *.Mask F.SilkS)
-      (net 5 GND))
-    (pad 6 thru_hole oval (at 3.4991 1.13746 270) (size 1.55 1) (drill oval 1.15 0.5) (layers *.Cu *.Mask F.SilkS)
+    (pad 6 thru_hole circle (at -2.5009 -1.56254 270) (size 1.25 1.25) (drill 0.85) (layers *.Cu *.Mask F.SilkS)
+      (net 5 GND))
+    (pad 6 thru_hole circle (at 2.4991 -1.56254 270) (size 1.25 1.25) (drill 0.85) (layers *.Cu *.Mask F.SilkS)
+      (net 5 GND))
+    (pad 6 thru_hole circle (at -3.5009 1.13746 270) (size 1.55 1.55) (drill 1.15) (layers *.Cu *.Mask F.SilkS)
+      (net 5 GND))
+    (pad 6 thru_hole circle (at 3.4991 1.13746 270) (size 1.55 1.55) (drill 1.15) (layers *.Cu *.Mask F.SilkS)
       (net 5 GND))
     (model ../../../../../home/lutz/kicad/DreErolf/10118194.wrl

Commit message: routed... at least for now
Parts:
- removed D8: D, Diodes_SMD:SOD-323
- removed IC1: L6205PD, BLDC:SOIC-20
- removed REF**1111111, REF**11111111111, REF**11111111112, REF**11111111113, REF**11111111114, REF**11111111121, REF**11111111122, REF**11111111123, REF**11111111124, REF**11111111131, REF**11111111132, REF**11111111133, REF**11111111134, REF**11111111141, REF**11111111142, REF**11111111143, REF**11111111144, REF**1111112, REF**1111113, REF**1111121, REF**1111122, REF**1111123, REF**1111131, REF**1111132, REF**1111133, REF**1111141, REF**1111142, REF**1111143, REF**1111151, REF**1111152, REF**1111153, REF**1111161, REF**1111162, REF**1111163, REF**1111171, REF**1111172, REF**1111173, REF**1111181, REF**1111182, REF**1111183: VIA-0.6, BLDC:VIA-0.6
- removed U5: MPU6000, Housings_DFN_QFN:QFN-24-1EP_4x4mm_Pitch0.5mm
- added C23: 1nF, Capacitors_SMD:C_0603, B.Cu at (119.0, 59.5)
- added C24: NA/100nF, Capacitors_SMD:C_0603, F.Cu at (122.5, 59.0)
- added D5: D_Small, Diodes_SMD:SOD-323, F.Cu at (133.0, 81.0)
- added D6: 3.3V, Diodes_SMD:SOD-323, F.Cu at (143.0, 64.0)
- added D7: 3.3V, Diodes_SMD:SOD-323, F.Cu at (143.0, 68.5)
- added JP1: OPEN, Resistors_SMD:R_0402, F.Cu at (130.0, 63.0)
- added Q1: Q_NMOS_DGS, BLDC:SOT1210, F.Cu at (106.0, 64.0)
- added Q2: Q_NMOS_DGS, BLDC:SOT1210, F.Cu at (106.0, 59.5)
- added Q3: Q_NMOS_DGS, BLDC:SOT1210, F.Cu at (111.0, 64.0)
- added Q4: Q_NMOS_DGS, BLDC:SOT1210, F.Cu at (111.0, 59.5)
- added Q5: Q_NMOS_DGS, BLDC:SOT1210, F.Cu at (116.0, 64.0)
- added Q6: Q_NMOS_DGS, BLDC:SOT1210, F.Cu at (116.0, 59.5)
- added Q7: 2N7002, TO_SOT_Packages_SMD:SOT-23, F.Cu at (120.5, 64.5)
- added R12: .01, Resistors_SMD:R_1210, B.Cu at (103.8, 57.2)
- added R13: 10R, Resistors_SMD:R_0603, F.Cu at (114.3, 69.5)
- added R14: 10R, Resistors_SMD:R_0603, F.Cu at (115.8, 69.5)
- added R15: NA/10kR, Resistors_SMD:R_0603, F.Cu at (121.0, 61.5)
- added R16: NA/10kR, Resistors_SMD:R_0603, F.Cu at (119.5, 61.5)
- added R17: 0R/50kR, Resistors_SMD:R_0603, F.Cu at (121.0, 59.0)
- added R18: NA/50kR, Resistors_SMD:R_0603, F.Cu at (119.5, 59.0)
- added U2: DRV8313, BLDC:SOIC-48, F.Cu at (112.5, 77.5)
- C1: value 220nF -> 100nF; moved to F.Cu
- C10, C12, C21, C3, C4, C5, C6, C7, C8, C9, D4, R5, U7: moved to F.Cu
- C11: value 100nF -> 2.2uF
- C17: value 2.2uF -> 100nF; moved to F.Cu
- C18, C19: value 2nF -> 100nF; moved to F.Cu
- C2: value 10nF -> 22nF; moved to F.Cu
- C20: value 100nF -> 10uF; footprint Capacitors_SMD:C_0603 -> Capacitors_ThroughHole:C_Radial_D5_L11_P2; moved to F.Cu
- C22: value 4.7uF -> 1nF; footprint Capacitors_SMD:C_0805 -> Capacitors_SMD:C_0603
- D1, D2: value D_Small -> 3.3V; moved to F.Cu
- P3: value CON_MOTOR -> CONN_01X03; footprint Terminal_Blocks:TerminalBlock_Pheonix_MPT-2.54mm_4pol -> Terminal_Blocks:TerminalBlock_Pheonix_MPT-2.54mm_3pol
- P7: footprint Connectors_Molex:Molex_KK-6410-04_04x2.54mm_Straight -> Terminal_Blocks:TerminalBlock_Pheonix_MPT-2.54mm_4pol
- R1: value 100 -> 10kR; moved to F.Cu
- R10, R11, R9: value .1 -> 10R; footprint Resistors_SMD:R_1206 -> Resistors_SMD:R_0603; moved to F.Cu
- R2: value NA -> 10kR; moved to F.Cu
- R3: value 0 -> 10kR; moved to F.Cu
- R4: value 10k -> 10kR; moved to F.Cu
- R6: value 10k -> 1R; moved to F.Cu
- R7: value 10k -> 10R; moved to F.Cu
- R8: value .1 -> .01; footprint Resistors_SMD:R_1206 -> Resistors_SMD:R_1210
- RP1: value 10k -> 20k; moved to F.Cu
- RP3: value 1k -> 10k; moved to F.Cu
- U1: value STM32F405R -> STM32F401CBUx; footprint Housings_QFP:TQFP-64_10x10mm_Pitch0.5mm -> Housings_DFN_QFN:QFN-48-1EP_7x7mm_Pitch0.5mm
- moved C22 55.0 mm to (102.3, 60.1), turned to 90 degrees
- moved C11 48.7 mm to (110.5, 84.5), turned to 270 degrees
- moved C20 45.5 mm to (104.5, 69.5), turned to 180 degrees
- moved C15 43.2 mm to (115.5, 84.5), turned to 270 degrees
- moved C16 43.2 mm to (117.0, 84.5), turned to 270 degrees
- moved C17 40.5 mm to (108.6, 71.5)
- moved D3 38.9 mm to (131.5, 52.5)
- moved R5 37.9 mm to (131.5, 55.5), turned to 270 degrees
- moved C7 37.3 mm to (134.0, 58.0), turned to 0 degrees
- moved R10 35.0 mm to (111.1, 69.5), turned to 270 degrees
- moved C14 34.8 mm to (121.5, 78.0), turned to 270 degrees
- moved R4 34.2 mm to (122.0, 75.0), turned to 90 degrees
- moved U7 32.9 mm to (126.0, 77.0), turned to 0 degrees
- moved R6 32.0 mm to (108.0, 84.5), turned to 270 degrees
- moved D4 31.5 mm to (133.0, 79.5), turned to 0 degrees
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Connections:
- net /OSC/OSC_IN renamed /OSC_IN
- net /OSC/OSC_OUT renamed /OSC_OUT
- C1 pad 1: Net-(C1-Pad1) -> /BOOT
- C1 pad 2: VPP -> GND
- C16 pad 1: VCC -> Net-(C16-Pad1)
- C17 pad 1: Net-(C17-Pad1) -> /DRV_OUT_1
- C17 pad 2: GND -> Net-(C17-Pad2)
- C18 pad 1: Net-(C18-Pad1) -> /DRV_OUT_2
- C18 pad 2: GND -> Net-(C18-Pad2)
- C19 pad 1: Net-(C19-Pad1) -> /DRV_OUT_3
- C19 pad 2: GND -> Net-(C19-Pad2)
- C22 pad 1: VPP -> GND
- C22 pad 2: GND -> Net-(C22-Pad2)
- D1 pad 1: Net-(D1-Pad1) -> /SENSE_V_3
- D1 pad 2: VPP -> GND
- D2 pad 1: Net-(C1-Pad1) -> /SENSE_V_2
- D2 pad 2: Net-(D1-Pad1) -> GND
- P1 pad 2: /CON_LED/LED_DATA -> /LED_MOSI
- P11 pad 1: /2CON/SIG_1 -> GND
- P11 pad 3: GND -> /PWM_2
- P12 pad 1: /2CON/SIG_2 -> GND
- P12 pad 3: GND -> /PWM_1
- P3 pad 1: /CON_MOTOR/C -> /DRV_OUT_3
- P3 pad 2: /CON_MOTOR/A -> /DRV_OUT_2
- P3 pad 3: /CON_MOTOR/B -> /DRV_OUT_1
- P4 pad 2: /USB/USB_DM -> /USB_D-
- P4 pad 3: /USB/USB_DP -> /USB_D+
- P5 pad 2: /SWDIO/NRST -> /NRST
- P5 pad 3: /SWDIO/SWDCLK -> /SWDCLK
- P5 pad 4: /SWDIO/SWDIO -> /SWDIO
- P6 pad 2: /HALL/HALL_W -> /HALL_W
- P6 pad 3: /HALL/HALL_V -> /HALL_V
- P6 pad 4: /HALL/HALL_U -> Net-(C24-Pad1)
- P6 pad 5: VCC -> +5V
- P7 pad 4: /Power/RX_TX_PWR_BOARD -> /COM_RX_TX_1
- R1 pad 1: Net-(C2-Pad2) -> /BOOT
- R1 pad 2: Net-(D1-Pad1) -> GND
- R10 pad 1: /driver/SENSE_A -> Net-(Q3-Pad2)
- R10 pad 2: GND -> Net-(R10-Pad2)
- R11 pad 1: /driver/SENSE_A -> Net-(Q4-Pad2)
- R11 pad 2: GND -> Net-(R11-Pad2)
- R2 pad 2: Net-(R2-Pad2) -> /DRV_NOCTW
- R3 pad 1: Net-(R2-Pad2) -> /NRST
- R3 pad 2: GND -> VCC
- R4 pad 2: /SWDIO/NRST -> /DRV_NFAULT
- R6 pad 1: Net-(C19-Pad1) -> Net-(R6-Pad1)
- R6 pad 2: /driver/EN_A -> GND
- R7 pad 1: Net-(C18-Pad1) -> Net-(Q1-Pad2)
- R7 pad 2: /driver/EN_B -> Net-(R7-Pad2)
- R8 pad 1: /driver/SENSE_B -> Net-(C22-Pad2)
- R9 pad 1: /driver/SENSE_B -> Net-(Q2-Pad2)
- R9 pad 2: GND -> Net-(R9-Pad2)
- RP1 pad 1: /CON_MOTOR/D -> /DRV_OUT_1
- RP1 pad 2: /CON_MOTOR/B -> /DRV_OUT_2
- RP1 pad 3: /CON_MOTOR/A -> /DRV_OUT_3
- RP1 pad 4: /CON_MOTOR/C -> VPP
- RP3 pad 1: /CUR_SENSE_4/OUT_4 -> /V_PP_SENSE
- RP3 pad 2: /CUR_SENSE_4/OUT_3 -> /SENSE_V_3
- RP3 pad 3: /CUR_SENSE_4/OUT_2 -> /SENSE_V_2
- RP3 pad 4: /CUR_SENSE_4/OUT_1 -> /SENSE_V_1
- U1 pad 10: (no net) -> /HALL_U
- U1 pad 11: /CON_LED/LED_DATA -> /HALL_V
- U1 pad 12: GND -> /HALL_W
- U1 pad 13: VCC -> /HALL_PWM
- U1 pad 14: /Power/RX_TX_PWR_BOARD -> /V_PP_SENSE
- U1 pad 15: /Power/RX_TX_PWR_BOARD -> /SENSE_V_3
- U1 pad 16: /2CON/SIG_2 -> /SENSE_V_2
- U1 pad 17: /2CON/SIG_1 -> /SENSE_V_1
- U1 pad 18: GND -> /CUR_SENSE_1
- U1 pad 19: VCC -> /DRV_L_C
- U1 pad 2: Net-(R5-Pad2) -> /DRV_NOCTW
- U1 pad 20: /IMU/nCS -> (no net)
- U1 pad 21: /IMU/SCK -> /DRV_DC_CAL
- U1 pad 22: /IMU/SDO -> Net-(C12-Pad1)
- U1 pad 23: /IMU/SDI -> GND
- U1 pad 24: /CUR_SENSE_4/OUT_1 -> VCC
- U1 pad 25: /CUR_SENSE_4/OUT_2 -> /DRV_ENABLE
- U1 pad 26: /CUR_SENSE_4/OUT_3 -> /DRV_L_A
- U1 pad 27: /CUR_SENSE_4/OUT_4 -> /DRV_L_B
- U1 pad 28: GND -> /LED_MOSI
- U1 pad 29: (no net) -> /DRV_H_A
- U1 pad 3: (no net) -> /DRV_NFAULT
- U1 pad 30: (no net) -> /DRV_H_B
- U1 pad 31: Net-(C12-Pad1) -> /DRV_H_C
- U1 pad 32: VCC -> /USB_D-
- U1 pad 33: (no net) -> /USB_D+
- U1 pad 34: (no net) -> /SWDIO
- U1 pad 35: (no net) -> GND
- U1 pad 36: (no net) -> VCC
- U1 pad 37: (no net) -> /SWDCLK
- U1 pad 38: (no net) -> Net-(R5-Pad2)
- U1 pad 39: (no net) -> /SPI_SCK
- U1 pad 4: (no net) -> /DRV_SPI_NCS
- U1 pad 40: (no net) -> /SPI_MISO
- U1 pad 41: /HALL/HALL_W -> /SPI_MOSI
- U1 pad 42: /HALL/HALL_V -> /BOOT
- U1 pad 43: /HALL/HALL_U -> /COM_RX_TX_1
- U1 pad 44: /USB/USB_DM -> /BOOT
- U1 pad 45: /USB/USB_DP -> /PWM_1
- U1 pad 46: /SWDIO/SWDIO -> /PWM_2
- U1 pad 47: Net-(C17-Pad1) -> GND
- U1 pad 49: /SWDIO/SWDCLK -> GND
- U1 pad 7: /SWDIO/NRST -> /NRST
- U1 pad 8: /driver/SENSE_A -> GND
- U1 pad 9: /driver/SENSE_B -> VCC
Routing:
- net /HALL_PWM: track 0.00 -> 65.8 mm, vias 0 -> 4
- net /HALL_U: track 0.00 -> 58.4 mm, vias 0 -> 2
- net Net-(D4-Pad2): track 3.40 -> 57.8 mm, vias 1 -> 2
- net Net-(C22-Pad2): track 0.00 -> 49.8 mm, vias 0 -> 13
- net /DRV_DC_CAL: track 0.00 -> 49.5 mm, vias 0 -> 4
- net /DRV_H_A: track 0.00 -> 48.7 mm, vias 0 -> 2
- net /DRV_ENABLE: track 0.00 -> 48.3 mm, vias 0 -> 2
- net /DRV_L_A: track 0.00 -> 46.4 mm, vias 0 -> 2
- net /DRV_H_B: track 0.00 -> 46.0 mm, vias 0 -> 2
- net /DRV_L_B: track 0.00 -> 44.8 mm, vias 0 -> 2
- net +5V: track 54.4 -> 99.0 mm, vias 3 -> 1
- net /SPI_MOSI: track 0.00 -> 44.2 mm, vias 0 -> 2
- net GND: track 25.7 -> 69.5 mm, vias 16 -> 35
- net /DRV_H_C: track 0.00 -> 43.7 mm, vias 0 -> 2
- net /DRV_L_C: track 0.00 -> 43.3 mm, vias 0 -> 4
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- added copper zone on F.Cu, net /DRV_OUT_1
- added copper zone on F.Cu, net /DRV_OUT_2
- added copper zone on F.Cu, net /DRV_OUT_3
- added copper zone on B.Cu, net Net-(C22-Pad2)
- added copper zone on F.Cu, net Net-(C22-Pad2)
- removed copper zone on F.Cu, net /CON_MOTOR/A
- removed copper zone on F.Cu, net /CON_MOTOR/B
- removed copper zone on F.Cu, net /CON_MOTOR/C
- removed copper zone on F.Cu, net /CON_MOTOR/D
- removed copper zone on B.Cu, net /driver/SENSE_A
- removed copper zone on F.Cu, net /driver/SENSE_A
- removed copper zone on B.Cu, net /driver/SENSE_B
- removed copper zone on F.Cu, net /driver/SENSE_B
Other:
- board size 47 x 39 mm -> 50 x 40 mm
- rule trace_min: 0.15 -> 0.1499

Commit message: some sugar
Routing:
- net Net-(D4-Pad2): track 57.8 -> 47.0 mm, vias 2 -> 4
- net /NRST: track 22.1 -> 19.8 mm
- net +5V: track 99.0 -> 97.8 mm, vias 1 -> 2
- net /OSC_OUT: track 11.0 -> 10.4 mm
- net /HALL_PWM: track 65.8 -> 66.3 mm

Commit message: well... actually we dont need those thwo parts since the bootloader can be entered from flash software
Parts:
- C1: value 100nF -> NA/100nF
- R1: value 10kR -> NA/10kR
Changed lines of the file:
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@@
   (general
     (links 241)
-    (no_connects 2)
+    (no_connects 0)
     (area 99.924999 49.924999 150.075001 90.075001)
     (thickness 1.6)
@@
       (effects (font (size 1 1) (thickness 0.15)))
     )
-    (fp_text value 100nF (at 0 1.9 180) (layer F.Fab)
+    (fp_text value NA/100nF (at 0 1.9 180) (layer F.Fab)
       (effects (font (size 1 1) (thickness 0.15)))
     )
@@
       (effects (font (size 1 1) (thickness 0.15)))
     )
-    (fp_text value 10kR (at 0 1.9 180) (layer F.Fab)
-      (effects (font (size 1 1) (thickness 0.15)))
-    )
+    (fp_text value NA/10kR (at 0 1.9 180) (layer F.Fab)
+      (effects (font (size 1 1) (thickness 0.15)))
+    )
