File: bldc-controller.kicad_pcb (KiCad board)
At the start: 2 copper layers, 50 x 40 mm, 76 parts, among them P1 CON_LED, P10 MOUNTING, P11 CONN_01X03, P12 CONN_01X03, P2 MOUNTING, P3 CONN_01X03, P4 USB_OTG, P5 CON_SWD, P6 CON_HALL, P7 CON_PWR_BRD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

Commit message: even though Im pretty sure that resistor is actually not needed Id like to play safe and have it anyway
Parts:
- R1: value NA/10kR -> 10kR
Changed lines of the file:
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@@
       (effects (font (size 1 1) (thickness 0.15)))
     )
-    (fp_text value NA/10kR (at 0 1.9 180) (layer F.Fab)
+    (fp_text value 10kR (at 0 1.9 180) (layer F.Fab)
       (effects (font (size 1 1) (thickness 0.15)))
     )
