File: bldc-controller.kicad_pcb (KiCad board)
At the start: 2 copper layers, 50 x 40 mm, 76 parts, among them P1 CON_LED, P10 MOUNTING, P11 CONN_01X03, P12 CONN_01X03, P2 MOUNTING, P3 CONN_01X03, P4 USB_OTG, P5 CON_SWD, P6 CON_HALL, P7 CON_PWR_BRD, P8 MOUNTING, P9 MOUNTING, Q1 Q_NMOS_DGS, Q2 Q_NMOS_DGS, Q3 Q_NMOS_DGS, Q4 Q_NMOS_DGS, Q5 Q_NMOS_DGS, Q6 Q_NMOS_DGS, Q7 2N7002, U1 STM32F401CBUx, U2 DRV8313, U7 LD1117S33TR, Y1 Crystal

Commit message: corrected order version
Routing:
- net Net-(D4-Pad2): track 47.0 -> 47.5 mm

Commit message: blubb
Parts:
- renumbered P3 to ?, P7 to ?, P4 to ?, U1 to ?, P6 to ?, P5 to ?, P10 to ?, P8 to ?, P2 to ?, P9 to ?, P1 to LEDs, P12 to SRV_1, P11 to SRV_2
Routing:
- net GND: track 69.5 -> 71.0 mm
- net /SWDCLK: track 20.2 -> 21.0 mm
Other:
- board text added: "5V"
- board text added: "GND"
- board text added: "HU"
- board text added: "HV"
- board text added: "HW"
- board text added: "RX/TX"
- board text added: "U"
- board text added: "V"
- board text added: "VPP"
- board text added: "W"

Commit message: some sugar coating and updated gerbers
Other:
- board text added: "LED_SIG"
Changed lines of the file:
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@@
     (area 99.924999 49.924999 150.075001 90.075001)
     (thickness 1.6)
-    (drawings 18)
+    (drawings 21)
     (tracks 1123)
     (zones 0)
@@
   (page A4)
   (layers
-    (0 F.Cu signal)
-    (31 B.Cu signal)
+    (0 F.Cu signal hide)
+    (31 B.Cu signal hide)
     (32 B.Adhes user hide)
     (33 F.Adhes user hide)
@@
     )
   )
+  (gr_text LED_SIG (at 137.55 82.5 90) (layer B.SilkS)
+    (effects (font (size 1 1) (thickness 0.25)) (justify mirror))
+  )
+  (gr_text 5V (at 135 84.15 90) (layer B.SilkS)
+    (effects (font (size 1 1) (thickness 0.25)) (justify mirror))
+  )
+  (gr_text GND (at 140.1 84 90) (layer B.SilkS)
+    (effects (font (size 1 1) (thickness 0.25)) (justify mirror))
+  )
   (gr_text RX/TX (at 121.5 83.25 90) (layer B.SilkS)
