File: bldc-controller.sch (KiCad schematic (older format))
At the start: 14 parts

Commit message: blubb
Parts:
- removed U?: STM32F405R, TQFP64, symbol STM32F405R
- added U1: STM32F405R, Housings_QFP:TQFP-64_10x10mm_Pitch0.5mm, symbol STM32F405R
- C10, C12, C17, C3, C4, C5, C6, C7: renamed from C?; footprint (none) -> Capacitors_SMD:C_0603
- D3: renamed from D?; footprint (none) -> LEDs:LED_0805
- R2, R3, R4, R5: renamed from R?; footprint (none) -> Resistors_SMD:R_0603
Connections:
- net COM_RX_TX_1: now also U1.14 (PA0/WKUP/USART2_CTS/UART4_TX/TIM2_CH1_ETR/TIM5_CH1/TIM8_ETR), U1.15 (PA1/USART2_RTS/UART4_RX/TIM5_CH2/TIMM2_CH2)
- net COM_RX_TX_2: now also U1.16 (PA2/USART2_TX/TIM5_CH3/TIM9_CH1/TIM2_CH3), U1.17 (PA3/USART2_RX/TIM5_CH4/TIM9_CH2/TIM2_CH4/OTG_HS_ULPI_D0)
- net GND: now also U1.12 (VSSA), U1.18 (VSS), U1.28 (PB2/BOOT1), U1.63 (VSS)
- net IMU_SPI_CS: now also U1.20 (PA4/SPI1_NSS/SPI3_NSS/USART2_CK/OTG_HS_SOF/I2S3_WS)
- net IMU_SPI_MISO: now also U1.22 (PA6/SPI1_MISO/TIM8_BKIN/TIM13_CH1/TIM3_CH1/TIM1_BKIN)
- net IMU_SPI_MOSI: now also U1.23 (PA7/SPI1_MOSI/TIM8_CH1N/TIM14_CH1/TIM3_CH2/TIM1_CH1N)
- net IMU_SPI_SCK: now also U1.21 (PA5/SPI1_SCK/OTG_HS_ULPI_CK/TIM2_CH1_ETR/TIM8_CHIN)
- net LED_MOSI: now also U1.11 (PC3/SPI2_MOSI/I2S2_SD/OTG_HS_ULPI_NXT)
- net NRST: now also U1.7 (NRST)
- net OSC_IN: now also U1.5 (PH0/OSC_IN)
- net OSC_OUT: now also U1.6 (PH1/OSC_OUT)
- net PWM_A_1: now also U1.58 (PB6/I2C1_SCL/TIM4_CH1/CAN2_TX/USART1_TX)
- net PWM_A_2: now also U1.59 (PB7/I2C1_SDA/FSMC_NL/USART1_RX/TIM4_CH2)
- net PWM_B_1: now also U1.61 (PB8/TIM4_CH3/SDIO_D4/TIM10_CH1/I2C1_SCL/CAN1_RX)
- net PWM_B_2: now also U1.62 (PB9/SPI2_NSS/I2S2_WS/TIM4_CH4/TIM11_CH1/SDIO_D5/I2C1_SDA/CAN1_TX)
- net PWM_EN_A: now also U1.56 (PB4/NJTRST/SPI3_MISO/TIM3_CH1/SPI1_MISO/I2S3ext_SD)
- net PWM_EN_B: now also U1.57 (PB5/I2C1_SMBA/CAN2_RX/OTG_HS_ULPI_D7/TIM3_CH2/SPI1_MOSI/SPI3_MOSI/I2S3_SD)
- net SENSE_CUR_A: now also U1.8 (PC0/OTG_HS_ULPI_STP)
- net SENSE_CUR_B: now also U1.9 (PC1)
- net SWDCLK: now also U1.49 (PA14/JTCK/SWCLK)
- net SWDIO: now also U1.46 (PA13/JTMS/SWDIO)
- net UART_LIDAR_RX: now also U1.38 (PC7/I2S3_MCK/TIM8_CH2/SDIO_D7/USART6_RX/TIM3_CH2)
- net UART_LIDAR_TX: now also U1.37 (PC6/I2S2_MCK/TIM8_CH1/SDIO_D6/USART6_TX/TIM3_CH1)
- net USB_DM: now also U1.44 (PA11/USART1_CTS/CAN1_RX/TIM1_CH4_/OTG_FS_DM)
- net USB_DP: now also U1.45 (PA12/USART1_RTS/CAN1_TX/TIM1_ETR/OTG_FS_DP)
- net VCC: now also U1.1 (VBAT), U1.13 (VDDA), U1.19 (VDD), U1.32 (VDD), U1.48 (VDD), U1.64 (VDD)
- net at R5.2: now also U1.2 (PC13)
- net at C12.1: now also U1.31 (VCAP_1)
- net at C17.1: now also U1.47 (VCAP_2)
- net at R2.2, R3.1: now also U1.60 (BOOT0)
- new net HALL_U: U1.43 (PA10/USART1_RX/TIM1_CH3/OTG_FS_ID)
- new net HALL_V: U1.42 (PA9/USART1_TX/TIM1_CH2/I2C3_SMBA)
- new net HALL_W: U1.41 (PA8/MCO1/USART1_CK/TIM1_CH1/I2C3_SCL/OTG_FS_SOF)
- new net LIDAR_MOTOR_EN: U1.39 (PC8/TIM8_CH3/SDIO_D0/TIM3_CH3/USART6_CK)
- new net SENSE_V_A_1: U1.24 (PC4)
- new net SENSE_V_A_2: U1.25 (PC5)
- new net SENSE_V_B_1: U1.26 (PB0/TIM3_CH3/TIM8_CH2N/OTG_HS_ULPI_D1/TIM1_CH2N)
- new net SENSE_V_B_2: U1.27 (PB1/TIM3_CH4/TIM8_CH3N/OTG_HS_ULPI_D2/OTG_HS_INTN/TIM1_CH3N)
- no-connect marks 1 -> 17
Other:
- moved on the sheet: D3, R5

Commit message: routed
Connections:
- net PWM_A_1: now also U1.61 (PB8/TIM4_CH3/SDIO_D4/TIM10_CH1/I2C1_SCL/CAN1_RX); no longer U1.58 (PB6/I2C1_SCL/TIM4_CH1/CAN2_TX/USART1_TX)
- net PWM_A_2: now also U1.62 (PB9/SPI2_NSS/I2S2_WS/TIM4_CH4/TIM11_CH1/SDIO_D5/I2C1_SDA/CAN1_TX); no longer U1.59 (PB7/I2C1_SDA/FSMC_NL/USART1_RX/TIM4_CH2)
- net PWM_B_1: now also U1.59 (PB7/I2C1_SDA/FSMC_NL/USART1_RX/TIM4_CH2); no longer U1.61 (PB8/TIM4_CH3/SDIO_D4/TIM10_CH1/I2C1_SCL/CAN1_RX)
- net PWM_B_2: now also U1.58 (PB6/I2C1_SCL/TIM4_CH1/CAN2_TX/USART1_TX); no longer U1.62 (PB9/SPI2_NSS/I2S2_WS/TIM4_CH4/TIM11_CH1/SDIO_D5/I2C1_SDA/CAN1_TX)
- net COM_RX_TX_2: no longer names the net of U1.16 (PA2/USART2_TX/TIM5_CH3/TIM9_CH1/TIM2_CH3)
- net COM_RX_TX_2: no longer U1.17 (PA3/USART2_RX/TIM5_CH4/TIM9_CH2/TIM2_CH4/OTG_HS_ULPI_D0)
- net LIDAR_MOTOR_EN: no longer names the net of U1.39 (PC8/TIM8_CH3/SDIO_D0/TIM3_CH3/USART6_CK)
- net UART_LIDAR_RX: no longer names the net of U1.38 (PC7/I2S3_MCK/TIM8_CH2/SDIO_D7/USART6_RX/TIM3_CH2)
- net UART_LIDAR_TX: no longer names the net of U1.37 (PC6/I2S2_MCK/TIM8_CH1/SDIO_D6/USART6_TX/TIM3_CH1)
- no-connect marks 17 -> 22
Changed lines of the file:
@@
 $Descr A4 11693 8268
 encoding utf-8
-Sheet 1 13
+Sheet 1 12
 Title ""
 Date ""
@@
 Wire Wire Line
 	3300 7000 3250 7000
+Text Label 3300 7500 0    60   ~ 0
+PWM_EN_A
 Text Label 3300 7400 0    60   ~ 0
-PWM_EN_A
-Text Label 3300 7500 0    60   ~ 0
 PWM_EN_B
 Wire Wire Line
@@
 NRST
 Connection ~ 1450 2050
+Text Label 8850 2550 0    60   ~ 0
+PWM_A_1
+Text Label 8850 2650 0    60   ~ 0
+PWM_A_2
+Text Label 8850 2450 0    60   ~ 0
+PWM_B_1
 Text Label 8850 2350 0    60   ~ 0
-PWM_A_1
-Text Label 8850 2450 0    60   ~ 0
-PWM_A_2
-Text Label 8850 2550 0    60   ~ 0
-PWM_B_1
-Text Label 8850 2650 0    60   ~ 0
 PWM_B_2
 Wire Wire Line
@@
 Text Label 1750 3650 2    60   ~ 0
 COM_RX_TX_1
-Text Label 1750 3850 2    60   ~ 0
-COM_RX_TX_2
-Wire Wire Line
-	1750 3850 1800 3850
 Wire Wire Line
 	1800 3650 1750 3650
@@
 F0 "Power" 60
 F1 "Power.sch" 60
-F2 "RX_PWR_BOARD" I R 5600 7050 60
-F3 "TX_PWR_BOARD" I R 5600 7150 60
+F2 "RX_TX_PWR_BOARD" I R 5600 7200 60
 $EndSheet
 Text Label 1750 4150 2    60   ~ 0
@@
 Wire Wire Line
 	1750 3750 1750 3650
-Wire Wire Line
-	1750 3850 1750 3950
-Wire Wire Line
-	1750 3950 1800 3950
 Wire Wire Line
 	8850 3650 8800 3650
@@
 Wire Wire Line
 	1800 4050 1750 4050
-Text Label 8850 4150 0    60   ~ 0
-UART_LIDAR_TX
-Text Label 8850 4250 0    60   ~ 0
-UART_LIDAR_RX
-Wire Wire Line
-	8850 4250 8800 4250
-Wire Wire Line
-	8800 4150 8850 4150
 Text Label 8850 3950 0    60   ~ 0
 SENSE_V_A_1
@@
 Wire Wire Line
 	10600 3100 10650 3100
-$Sheet
-S 10300 5800 850  300
-U 57ACFC7C
-F0 "CON_LIDAR" 60
-F1 "CON_LIDAR.sch" 60
-F2 "LIDAR_MOTOR_EN" I L 10300 5850 60
-F3 "LIDAR_RX" I L 10300 5950 60
-F4 "LIDAR_TX" I L 10300 6050 60
-$EndSheet
-Text Label 10250 5950 2    60   ~ 0
-UART_LIDAR_RX
-Text Label 10250 6050 2    60   ~ 0
-UART_LIDAR_TX
-Wire Wire Line
-	10250 6050 10300 6050
-Wire Wire Line
-	10250 5950 10300 5950
-Text Label 8850 4350 0    60   ~ 0
-LIDAR_MOTOR_EN
-Wire Wire Line
-	8850 4350 8800 4350
-Text Label 10250 5850 2    60   ~ 0
-LIDAR_MOTOR_EN
-Wire Wire Line
-	10250 5850 10300 5850
 $Sheet
 S 2350 6350 500  400
@@
 F1 "Holes.sch" 60
 $EndSheet
-Text Label 5700 7050 0    60   ~ 0
+Text Label 5700 7200 0    60   ~ 0
 COM_RX_TX_1
-Text Label 5700 7150 0    60   ~ 0
-COM_RX_TX_2
-Wire Wire Line
-	5700 7150 5600 7150
-Wire Wire Line
-	5600 7050 5700 7050
+Wire Wire Line
+	5600 7200 5700 7200
 Text Label 700  5950 0    60   ~ 0
 IMU_SPI_CS
@@
 	1    0    0    -1
 $EndComp
+NoConn ~ 8800 4150
+NoConn ~ 8800 4250
+NoConn ~ 8800 4350
+NoConn ~ 1800 3950
+NoConn ~ 1800 3850
 $EndSCHEMATC

Commit message: fertig?
Connections:
- net PWM_1: now reaches U1.16 (PA2/USART2_TX/TIM5_CH3/TIM9_CH1/TIM2_CH3)
- net PWM_2: now reaches U1.17 (PA3/USART2_RX/TIM5_CH4/TIM9_CH2/TIM2_CH4/OTG_HS_ULPI_D0)
- no-connect marks 22 -> 20
Changed lines of the file:
@@
 $Descr A4 11693 8268
 encoding utf-8
-Sheet 1 12
+Sheet 1 13
 Title ""
 Date ""
@@
 NoConn ~ 8800 4250
 NoConn ~ 8800 4350
-NoConn ~ 1800 3950
-NoConn ~ 1800 3850
+Text Label 1750 3850 2    60   ~ 0
+PWM_1
+Text Label 1750 3950 2    60   ~ 0
+PWM_2
+Wire Wire Line
+	1750 3850 1800 3850
+Wire Wire Line
+	1800 3950 1750 3950
+$Sheet
+S 10650 3450 500  250
+U 57B721E0
+F0 "2CON" 60
+F1 "2CON.sch" 60
+F2 "SIG_1" I L 10650 3500 60
+F3 "SIG_2" I L 10650 3600 60
+$EndSheet
+Text Label 10600 3600 2    60   ~ 0
+PWM_1
+Text Label 10600 3500 2    60   ~ 0
+PWM_2
+Wire Wire Line
+	10600 3600 10650 3600
+Wire Wire Line
+	10650 3500 10600 3500
 $EndSCHEMATC

Commit message: updated stuff
Parts:
- removed C17: 2.2uF, Capacitors_SMD:C_0603, symbol C
- removed R4: 10k, Resistors_SMD:R_0603, symbol R_Small
- removed U1: STM32F405R, Housings_QFP:TQFP-64_10x10mm_Pitch0.5mm, symbol STM32F405R
- added JP?: OPEN, symbol JUMPER
- added U?: STM32F401CBUx, UFQFPN48, symbol STM32F401CBUx
- R3: value 0 -> 10kR
Connections:
- net COM_RX_TX_1: now also U?.39 (PB3/I2C2_SDA/I2S3_CK/SPI1_SCK/SPI3_SCK/SYS_JTDO-SWO/TIM2_CH2), U?.40 (PB4/I2C3_SDA/I2S3_ext_SD/SPI1_MISO/SPI3_MISO/SYS_JTRST/TIM3_CH1)
- net GND: now also U?.23 (VSS), U?.35 (VSS), U?.47 (VSS), U?.49 (VSS), U?.8 (VSSA)
- net HALL_U: now also U?.41 (PB5/I2C1_SMBA/I2S3_SD/SPI1_MOSI/SPI3_MOSI/TIM3_CH2)
- net HALL_V: now also U?.42 (PB6/I2C1_SCL/TIM4_CH1/USART1_TX)
- net HALL_W: now also U?.43 (PB7/I2C1_SDA/TIM4_CH2/USART1_RX)
- net NRST: now also R2.2, R3.1, U?.7 (NRST)
- net PWM_1: now also U?.12 (ADC1_IN2/TIM2_CH3/TIM5_CH3/TIM9_CH1/USART2_TX/PA2)
- net PWM_2: now also U?.13 (ADC1_IN3/TIM2_CH4/TIM5_CH4/TIM9_CH2/USART2_RX/PA3)
- net SWDCLK: now also U?.37 (SYS_JTCK-SWCLK/PA14)
- net SWDIO: now also U?.34 (SYS_JTMS-SWDIO/PA13)
- net USB_DM: now also U?.32 (ADC1_EXTI11/TIM1_CH4/USART1_CTS/USART6_TX/USB_OTG_FS_DM/PA11)
- net USB_DP: now also U?.33 (TIM1_ETR/USART1_RTS/USART6_RX/USB_OTG_FS_DP/PA12)
- net VCC: now also JP?.1, U?.1 (VBAT), U?.24 (VDD), U?.36 (VDD), U?.48 (VDD), U?.9 (VREF+)
- net at C12.1: now also U?.22 (VCAP1)
- net at R5.2: now also U?.38 (ADC1_EXTI15/I2S3_WS/SPI1_NSS/SPI3_NSS/SYS_JTDI/TIM2_CH1/TIM2_ETR/PA15)
- new net: JP?.2, U?.44 (BOOT0)
- new net CUR_SENSE_1: U?.18 (PB0/ADC1_IN8/TIM1_CH2N/TIM3_CH3)
- new net CUR_SENSE_2: U?.19 (PB1/ADC1_IN9/TIM1_CH3N/TIM3_CH4)
- new net DRV_H_A: U?.29 (I2C3_SCL/RCC_MCO_1/TIM1_CH1/USART1_CK/USB_OTG_FS_SOF/PA8)
- new net DRV_H_B: U?.30 (I2C3_SMBA/TIM1_CH2/USART1_TX/USB_OTG_FS_VBUS/PA9)
- new net DRV_H_C: U?.31 (TIM1_CH3/USART1_RX/USB_OTG_FS_ID/PA10)
- new net DRV_L_A: U?.26 (PB13/I2S2_CK/SPI2_SCK/TIM1_CH1N)
- new net DRV_L_B: U?.27 (PB14/I2S2_ext_SD/SPI2_MISO/TIM1_CH2N)
- new net DRV_L_C: U?.28 (PB15/ADC1_EXTI15/I2S2_SD/RTC_REFIN/SPI2_MOSI/TIM1_CH3N)
- new net DRV_NFAULT: U?.46 (PB9/I2C1_SDA/I2S2_WS/SPI2_NSS/TIM11_CH1/TIM4_CH4)
- new net DRV_NOCTW: U?.45 (PB8/I2C1_SCL/TIM10_CH1/TIM4_CH3)
- new net DRV_SPI_NCS: U?.21 (PB10/I2C2_SCL/I2S2_CK/SPI2_SCK/TIM2_CH3)
- new net OSC/OSC_IN: U?.5 (PH0/RCC_OSC_IN)
- new net OSC/OSC_OUT: U?.6 (PH1/RCC_OSC_OUT)
- new net SENSE_V_1: U?.10 (ADC1_IN0/SYS_WKUP/TIM2_CH1/TIM2_ETR/TIM5_CH1/USART2_CTS/PA0)
- new net SENSE_V_2: U?.11 (ADC1_IN1/TIM2_CH2/TIM5_CH2/USART2_RTS/PA1)
- new net SENSE_V_3: U?.14 (ADC1_IN4/I2S3_WS/SPI1_NSS/SPI3_NSS/USART2_CK/PA4)
- new net SPI_MISO: U?.16 (ADC1_IN6/SPI1_MISO/TIM1_BKIN/TIM3_CH1/PA6)
- new net SPI_MOSI: U?.17 (ADC1_IN7/SPI1_MOSI/TIM1_CH1N/TIM3_CH2/PA7)
- new net SPI_SCK: U?.15 (ADC1_IN5/SPI1_SCK/TIM2_CH1/TIM2_ETR/PA5)
- no-connect marks 20 -> 3
Other:
- moved on the sheet: C10, C12, C3, C4, C5, C6, C7, D3, R5

Commit message: i think im good with the schematics
Connections:
- net COM_RX_TX_1: now also U?.42 (PB6/I2C1_SCL/TIM4_CH1/USART1_TX), U?.43 (PB7/I2C1_SDA/TIM4_CH2/USART1_RX); no longer U?.39 (PB3/I2C2_SDA/I2S3_CK/SPI1_SCK/SPI3_SCK/SYS_JTDO-SWO/TIM2_CH2), U?.40 (PB4/I2C3_SDA/I2S3_ext_SD/SPI1_MISO/SPI3_MISO/SYS_JTRST/TIM3_CH1)
- net CUR_SENSE_2: now also U?.14 (ADC1_IN4/I2S3_WS/SPI1_NSS/SPI3_NSS/USART2_CK/PA4); no longer U?.19 (PB1/ADC1_IN9/TIM1_CH3N/TIM3_CH4)
- net DRV_L_C: now also U?.19 (PB1/ADC1_IN9/TIM1_CH3N/TIM3_CH4); no longer U?.28 (PB15/ADC1_EXTI15/I2S2_SD/RTC_REFIN/SPI2_MOSI/TIM1_CH3N)
- net DRV_NFAULT: now also U?.3 (PC14/RCC_OSC32_IN); no longer U?.46 (PB9/I2C1_SDA/I2S2_WS/SPI2_NSS/TIM11_CH1/TIM4_CH4)
- net DRV_NOCTW: now also U?.2 (PC13/ANTI_TAMP/RTC_AF1); no longer U?.45 (PB8/I2C1_SCL/TIM10_CH1/TIM4_CH3)
- net DRV_SPI_NCS: now also U?.4 (PC15/ADC1_EXTI15/RCC_OSC32_OUT); no longer U?.21 (PB10/I2C2_SCL/I2S2_CK/SPI2_SCK/TIM2_CH3)
- net HALL_U: now also U?.10 (ADC1_IN0/SYS_WKUP/TIM2_CH1/TIM2_ETR/TIM5_CH1/USART2_CTS/PA0); no longer U?.41 (PB5/I2C1_SMBA/I2S3_SD/SPI1_MOSI/SPI3_MOSI/TIM3_CH2)
- net HALL_V: now also U?.11 (ADC1_IN1/TIM2_CH2/TIM5_CH2/USART2_RTS/PA1); no longer U?.42 (PB6/I2C1_SCL/TIM4_CH1/USART1_TX)
- net HALL_W: now also U?.12 (ADC1_IN2/TIM2_CH3/TIM5_CH3/TIM9_CH1/USART2_TX/PA2); no longer U?.43 (PB7/I2C1_SDA/TIM4_CH2/USART1_RX)
- net LED_MOSI: now also U?.28 (PB15/ADC1_EXTI15/I2S2_SD/RTC_REFIN/SPI2_MOSI/TIM1_CH3N)
- net PWM_1: now also U?.45 (PB8/I2C1_SCL/TIM10_CH1/TIM4_CH3); no longer U?.12 (ADC1_IN2/TIM2_CH3/TIM5_CH3/TIM9_CH1/USART2_TX/PA2)
- net PWM_2: now also U?.46 (PB9/I2C1_SDA/I2S2_WS/SPI2_NSS/TIM11_CH1/TIM4_CH4); no longer U?.13 (ADC1_IN3/TIM2_CH4/TIM5_CH4/TIM9_CH2/USART2_RX/PA3)
- net SENSE_V_1: now also U?.15 (ADC1_IN5/SPI1_SCK/TIM2_CH1/TIM2_ETR/PA5); no longer U?.10 (ADC1_IN0/SYS_WKUP/TIM2_CH1/TIM2_ETR/TIM5_CH1/USART2_CTS/PA0)
- net SENSE_V_2: now also U?.16 (ADC1_IN6/SPI1_MISO/TIM1_BKIN/TIM3_CH1/PA6); no longer U?.11 (ADC1_IN1/TIM2_CH2/TIM5_CH2/USART2_RTS/PA1)
- net SENSE_V_3: now also U?.17 (ADC1_IN7/SPI1_MOSI/TIM1_CH1N/TIM3_CH2/PA7); no longer U?.14 (ADC1_IN4/I2S3_WS/SPI1_NSS/SPI3_NSS/USART2_CK/PA4)
- net SPI_MISO: now also U?.40 (PB4/I2C3_SDA/I2S3_ext_SD/SPI1_MISO/SPI3_MISO/SYS_JTRST/TIM3_CH1); no longer U?.16 (ADC1_IN6/SPI1_MISO/TIM1_BKIN/TIM3_CH1/PA6)
- net SPI_MOSI: now also U?.41 (PB5/I2C1_SMBA/I2S3_SD/SPI1_MOSI/SPI3_MOSI/TIM3_CH2); no longer U?.17 (ADC1_IN7/SPI1_MOSI/TIM1_CH1N/TIM3_CH2/PA7)
- net SPI_SCK: now also U?.39 (PB3/I2C2_SDA/I2S3_CK/SPI1_SCK/SPI3_SCK/SYS_JTDO-SWO/TIM2_CH2); no longer U?.15 (ADC1_IN5/SPI1_SCK/TIM2_CH1/TIM2_ETR/PA5)
- net OSC/OSC_IN renamed OSC_IN
- net OSC/OSC_OUT renamed OSC_OUT
- new net HALL_PWM: U?.13 (ADC1_IN3/TIM2_CH4/TIM5_CH4/TIM9_CH2/USART2_RX/PA3)
- no-connect marks 3 -> 1
