File: 2CON.sch (KiCad schematic (older format))
At the start: 2 parts, among them P11 CONN_01X03, P12 CONN_01X03

Commit message: routed... at least for now
Connections:
- net GND: now also P11.1 (P1), P12.1 (P1); no longer P11.3 (P3), P12.3 (P3)
- net SIG_1: now also P11.3 (P3); no longer P11.1 (P1)
- net SIG_2: now also P12.3 (P3); no longer P12.1 (P1)
Changed lines of the file:
@@
 $Descr A4 11693 8268
 encoding utf-8
-Sheet 13 12
+Sheet 10 12
 Title ""
 Date ""
@@
 F 3 "" H 1700 1050 50  0000 C CNN
 	1    1700 1050
-	1    0    0    -1
+	1    0    0    1
 $EndComp
 $Comp
@@
 F 3 "" H 1700 1450 50  0000 C CNN
 	1    1700 1450
-	1    0    0    -1
+	1    0    0    1
 $EndComp
 $Comp
-L GND #PWR051
+L GND #PWR037
 U 1 1 57B72381
 P 1400 1650
-F 0 "#PWR051" H 1400 1400 50  0001 C CNN
+F 0 "#PWR037" H 1400 1400 50  0001 C CNN
 F 1 "GND" H 1400 1500 50  0000 C CNN
 F 2 "" H 1400 1650 50  0000 C CNN
@@
 $EndComp
 $Comp
-L +5VA #PWR052
+L +5VA #PWR038
 U 1 1 57B723C7
 P 1300 750
-F 0 "#PWR052" H 1300 600 50  0001 C CNN
+F 0 "#PWR038" H 1300 600 50  0001 C CNN
 F 1 "+5VA" H 1300 890 50  0000 C CNN
 F 2 "" H 1300 750 50  0000 C CNN

Commit message: long forgotten commit of something I did half a year ago -.-
Parts:
- removed P11, P12: CONN_01X03, Pin_Headers:Pin_Header_Straight_1x03, symbol CONN_01X03
- added J1: Conn_02x03_Odd_Even, Connector_PinHeader_2.00mm:PinHeader_2x03_P2.00mm_Horizontal, symbol Connector_Generic:Conn_02x03_Odd_Even
Connections:
- wire segments 8 -> 10
Changed lines of the file:
@@
-EESchema Schematic File Version 2
-LIBS:bldc-controller-rescue
-LIBS:power
-LIBS:device
-LIBS:transistors
-LIBS:conn
-LIBS:linear
-LIBS:regul
-LIBS:74xx
-LIBS:cmos4000
-LIBS:adc-dac
-LIBS:memory
-LIBS:xilinx
-LIBS:microcontrollers
-LIBS:dsp
-LIBS:microchip
-LIBS:analog_switches
-LIBS:motorola
-LIBS:texas
-LIBS:intel
-LIBS:audio
-LIBS:interface
-LIBS:digital-audio
-LIBS:philips
-LIBS:display
-LIBS:cypress
-LIBS:siliconi
-LIBS:opto
-LIBS:atmel
-LIBS:contrib
-LIBS:valves
-LIBS:Power_Management
-LIBS:st-microelectronics
-LIBS:stm32
-LIBS:w_analog
-LIBS:mpu6000
+EESchema Schematic File Version 4
 LIBS:bldc-controller-cache
-EELAYER 25 0
+EELAYER 29 0
 EELAYER END
 $Descr A4 11693 8268
@@
 $EndDescr
 $Comp
-L CONN_01X03 P11
-U 1 1 57B7231D
-P 1700 1050
-F 0 "P11" H 1700 1250 50  0000 C CNN
-F 1 "CONN_01X03" V 1800 1050 50  0000 C CNN
-F 2 "Pin_Headers:Pin_Header_Straight_1x03" H 1700 1050 50  0001 C CNN
-F 3 "" H 1700 1050 50  0000 C CNN
-	1    1700 1050
+L Connector_Generic:Conn_02x03_Odd_Even J1
+U 1 1 5D353684
+P 2550 1150
+F 0 "J1" H 2600 825 50  0000 C CNN
+F 1 "Conn_02x03_Odd_Even" H 2600 916 50  0000 C CNN
+F 2 "Connector_PinHeader_2.00mm:PinHeader_2x03_P2.00mm_Horizontal" H 2550 1150 50  0001 C CNN
+F 3 "~" H 2550 1150 50  0001 C CNN
+	1    2550 1150
 	1    0    0    1
 $EndComp
 $Comp
-L CONN_01X03 P12
-U 1 1 57B7235F
-P 1700 1450
-F 0 "P12" H 1700 1650 50  0000 C CNN
-F 1 "CONN_01X03" V 1800 1450 50  0000 C CNN
-F 2 "Pin_Headers:Pin_Header_Straight_1x03" H 1700 1450 50  0001 C CNN
-F 3 "" H 1700 1450 50  0000 C CNN
-	1    1700 1450
-	1    0    0    1
-$EndComp
-$Comp
-L GND #PWR037
-U 1 1 57B72381
-P 1400 1650
-F 0 "#PWR037" H 1400 1400 50  0001 C CNN
-F 1 "GND" H 1400 1500 50  0000 C CNN
-F 2 "" H 1400 1650 50  0000 C CNN
-F 3 "" H 1400 1650 50  0000 C CNN
-	1    1400 1650
+L bldc-controller-rescue:GND #PWR0102
+U 1 1 5D35475B
+P 2250 1550
+F 0 "#PWR0102" H 2250 1300 50  0001 C CNN
+F 1 "GND" H 2250 1400 50  0000 C CNN
+F 2 "" H 2250 1550 50  0000 C CNN
+F 3 "" H 2250 1550 50  0000 C CNN
+	1    2250 1550
 	1    0    0    -1
 $EndComp
 $Comp
-L +5VA #PWR038
-U 1 1 57B723C7
-P 1300 750
-F 0 "#PWR038" H 1300 600 50  0001 C CNN
-F 1 "+5VA" H 1300 890 50  0000 C CNN
-F 2 "" H 1300 750 50  0000 C CNN
-F 3 "" H 1300 750 50  0000 C CNN
-	1    1300 750
+L bldc-controller-rescue:GND #PWR0103
+U 1 1 5D354AAB
+P 3000 1550
+F 0 "#PWR0103" H 3000 1300 50  0001 C CNN
+F 1 "GND" H 3000 1400 50  0000 C CNN
+F 2 "" H 3000 1550 50  0000 C CNN
+F 3 "" H 3000 1550 50  0000 C CNN
+	1    3000 1550
 	1    0    0    -1
 $EndComp
 Wire Wire Line
-	1300 750  1300 1450
+	3000 1550 3000 1050
 Wire Wire Line
-	1300 1050 1500 1050
+	3000 1050 2850 1050
 Wire Wire Line
-	1300 1450 1500 1450
-Connection ~ 1300 1050
+	2350 1050 2250 1050
 Wire Wire Line
-	1400 1150 1400 1650
+	2250 1050 2250 1550
+$Comp
+L bldc-controller-rescue:+5VA #PWR?
+U 1 1 5D3550F6
+P 2200 750
+AR Path="/5D3550F6" Ref="#PWR?"  Part="1"
+AR Path="/57B721E0/5D3550F6" Ref="#PWR0104"  Part="1"
+F 0 "#PWR0104" H 2200 600 50  0001 C CNN
+F 1 "+5VA" H 2200 890 50  0000 C CNN
+F 2 "" H 2200 750 50  0000 C CNN
+F 3 "" H 2200 750 50  0000 C CNN
+	1    2200 750
+	1    0    0    -1
+$EndComp
+$Comp
+L bldc-controller-rescue:+5VA #PWR?
+U 1 1 5D355436
+P 3050 750
+AR Path="/5D355436" Ref="#PWR?"  Part="1"
+AR Path="/57B721E0/5D355436" Ref="#PWR0105"  Part="1"
+F 0 "#PWR0105" H 3050 600 50  0001 C CNN
+F 1 "+5VA" H 3050 890 50  0000 C CNN
+F 2 "" H 3050 750 50  0000 C CNN
+F 3 "" H 3050 750 50  0000 C CNN
+	1    3050 750
+	1    0    0    -1
+$EndComp
 Wire Wire Line
-	1400 1550 1500 1550
+	3050 750  3050 1150
 Wire Wire Line
-	1400 1150 1500 1150
-Connection ~ 1400 1550
-Text HLabel 1100 950  0    60   Input ~ 0
+	3050 1150 2850 1150
+Wire Wire Line
+	2350 1150 2200 1150
+Wire Wire Line
+	2200 1150 2200 750
+Text HLabel 2150 1250 0    60   Input ~ 0
 SIG_1
-Text HLabel 1100 1350 0    60   Input ~ 0
+Wire Wire Line
+	2150 1250 2350 1250
+Text HLabel 3100 1250 2    60   Input ~ 0
 SIG_2
 Wire Wire Line
-	1100 1350 1500 1350
-Wire Wire Line
-	1100 950  1500 950
+	3150 1250 2850 1250
 $EndSCHEMATC
