File: CON_LED.sch (KiCad schematic (older format))
At the start: 1 part, among them P1 CON_LED

Commit message: blubb
Connections:
- net +5V renamed +5VA
Changed lines of the file:
@@
 $EndDescr
-$Comp
-L +5V #PWR046
-U 1 1 57ACE56F
-P 1250 800
-F 0 "#PWR046" H 1250 650 50  0001 C CNN
-F 1 "+5V" H 1250 940 50  0000 C CNN
-F 2 "" H 1250 800 50  0000 C CNN
-F 3 "" H 1250 800 50  0000 C CNN
-	1    1250 800
-	1    0    0    -1
-$EndComp
 $Comp
 L GND #PWR047
@@
 Wire Wire Line
 	1250 1050 1250 1100
+$Comp
+L +5VA #PWR?
+U 1 1 57B57C97
+P 1250 800
+F 0 "#PWR?" H 1250 650 50  0001 C CNN
+F 1 "+5VA" H 1250 940 50  0000 C CNN
+F 2 "" H 1250 800 50  0000 C CNN
+F 3 "" H 1250 800 50  0000 C CNN
+	1    1250 800
+	1    0    0    -1
+$EndComp
 $EndSCHEMATC

Commit message: fertig?
Parts:
- P1: footprint Connectors_Molex:Molex_KK-6410-03_03x2.54mm_Straight -> Pin_Headers:Pin_Header_Straight_1x03
Changed lines of the file:
@@
 $Descr A4 11693 8268
 encoding utf-8
-Sheet 9 12
+Sheet 9 13
 Title ""
 Date ""
@@
 F 0 "P1" H 1500 1150 50  0000 C CNN
 F 1 "CON_LED" V 1600 950 50  0000 C CNN
-F 2 "Connectors_Molex:Molex_KK-6410-03_03x2.54mm_Straight" H 1500 950 50  0001 C CNN
+F 2 "Pin_Headers:Pin_Header_Straight_1x03" H 1500 950 50  0001 C CNN
 F 3 "" H 1500 950 50  0000 C CNN
 	1    1500 950
@@
 	1250 1050 1250 1100
 $Comp
-L +5VA #PWR?
+L +5VA #PWR048
 U 1 1 57B57C97
 P 1250 800
-F 0 "#PWR?" H 1250 650 50  0001 C CNN
+F 0 "#PWR048" H 1250 650 50  0001 C CNN
 F 1 "+5VA" H 1250 940 50  0000 C CNN
 F 2 "" H 1250 800 50  0000 C CNN

Commit message: some sugar coating and updated gerbers
Connections:
- net +5VA: now also P1.3 (P3); no longer P1.1 (P1)
- net GND: now also P1.1 (P1); no longer P1.3 (P3)
Changed lines of the file:
@@
 F 3 "" H 1500 950 50  0000 C CNN
 	1    1500 950
-	1    0    0    -1
+	1    0    0    1
 $EndComp
 Wire Wire Line

Commit message: long forgotten commit of something I did half a year ago -.-
Parts:
- P1: footprint Pin_Headers:Pin_Header_Straight_1x03 -> Connector_PinHeader_2.54mm:PinHeader_1x03_P2.54mm_Vertical; symbol CONN_01X03 -> bldc-controller-rescue:CONN_01X03
Changed lines of the file:
@@
-EESchema Schematic File Version 2
-LIBS:bldc-controller-rescue
-LIBS:power
-LIBS:device
-LIBS:transistors
-LIBS:conn
-LIBS:linear
-LIBS:regul
-LIBS:74xx
-LIBS:cmos4000
-LIBS:adc-dac
-LIBS:memory
-LIBS:xilinx
-LIBS:microcontrollers
-LIBS:dsp
-LIBS:microchip
-LIBS:analog_switches
-LIBS:motorola
-LIBS:texas
-LIBS:intel
-LIBS:audio
-LIBS:interface
-LIBS:digital-audio
-LIBS:philips
-LIBS:display
-LIBS:cypress
-LIBS:siliconi
-LIBS:opto
-LIBS:atmel
-LIBS:contrib
-LIBS:valves
-LIBS:Power_Management
-LIBS:st-microelectronics
-LIBS:stm32
-LIBS:w_analog
-LIBS:mpu6000
+EESchema Schematic File Version 4
 LIBS:bldc-controller-cache
-EELAYER 25 0
+EELAYER 29 0
 EELAYER END
 $Descr A4 11693 8268
@@
 $EndDescr
 $Comp
-L GND #PWR035
+L bldc-controller-rescue:GND #PWR035
 U 1 1 57ACE583
 P 1250 1100
@@
 LED_DATA
 $Comp
-L CONN_01X03 P1
+L bldc-controller-rescue:CONN_01X03 P1
 U 1 1 57ACE598
 P 1500 950
 F 0 "P1" H 1500 1150 50  0000 C CNN
 F 1 "CON_LED" V 1600 950 50  0000 C CNN
-F 2 "Pin_Headers:Pin_Header_Straight_1x03" H 1500 950 50  0001 C CNN
+F 2 "Connector_PinHeader_2.54mm:PinHeader_1x03_P2.54mm_Vertical" H 1500 950 50  0001 C CNN
 F 3 "" H 1500 950 50  0000 C CNN
 	1    1500 950
@@
 	1250 1050 1250 1100
 $Comp
-L +5VA #PWR036
+L bldc-controller-rescue:+5VA #PWR036
 U 1 1 57B57C97
 P 1250 800
+AR Path="/57B57C97" Ref="#PWR036"  Part="1"
+AR Path="/57ACE4EA/57B57C97" Ref="#PWR036"  Part="1"
 F 0 "#PWR036" H 1250 650 50  0001 C CNN
 F 1 "+5VA" H 1250 940 50  0000 C CNN
