File: CUR_SENSE_4.sch (KiCad schematic (older format))
At the start: 7 parts

Commit message: blubb
Parts:
- removed D5, D6, D7, D9: 3V, Diodes_SMD:SOD-323, symbol D_Schottky_Small
Connections:
- wire segments 32 -> 22
Changed lines of the file:
@@
 Connection ~ 1500 1600
 $Comp
-L GND #PWR037
+L GND #PWR038
 U 1 1 57A226A1
 P 1550 1650
-F 0 "#PWR037" H 1550 1400 50  0001 C CNN
+F 0 "#PWR038" H 1550 1400 50  0001 C CNN
 F 1 "GND" H 1550 1500 50  0000 C CNN
 F 2 "" H 1550 1650 50  0000 C CNN
@@
 Connection ~ 1550 1600
 Wire Wire Line
-	2250 1200 2250 1050
-Wire Wire Line
 	2150 1050 2800 1050
-Wire Wire Line
-	2350 950  2350 1200
 Wire Wire Line
 	2150 950  2800 950
 Wire Wire Line
-	2450 850  2450 1200
-Wire Wire Line
 	2150 850  2800 850
-Wire Wire Line
-	2550 750  2550 1200
 Wire Wire Line
 	2150 750  2800 750
@@
 Text HLabel 2800 1050 2    60   Output ~ 0
 OUT_4
-Connection ~ 2250 1050
-Connection ~ 2350 950
-Connection ~ 2450 850
-Connection ~ 2550 750
-Wire Wire Line
-	2550 1500 2550 1400
-Wire Wire Line
-	2250 1500 2550 1500
-Wire Wire Line
-	2250 1500 2250 1400
-Wire Wire Line
-	2350 1400 2350 1500
-Connection ~ 2350 1500
-Wire Wire Line
-	2450 1400 2450 1500
-Connection ~ 2450 1500
-$Comp
-L GND #PWR038
-U 1 1 57A22B7D
-P 2400 1600
-F 0 "#PWR038" H 2400 1350 50  0001 C CNN
-F 1 "GND" H 2400 1450 50  0000 C CNN
-F 2 "" H 2400 1600 50  0000 C CNN
-F 3 "" H 2400 1600 50  0000 C CNN
-	1    2400 1600
-	1    0    0    -1
-$EndComp
-$Comp
-L D_Schottky_Small D5
-U 1 1 57A22C08
-P 2250 1300
-F 0 "D5" H 2200 1380 50  0000 L CNN
-F 1 "3V" H 2100 1250 50  0000 L CNN
-F 2 "Diodes_SMD:SOD-323" V 2250 1300 50  0001 C CNN
-F 3 "" V 2250 1300 50  0000 C CNN
-	1    2250 1300
-	0    1    1    0
-$EndComp
-$Comp
-L D_Schottky_Small D6
-U 1 1 57A22CDB
-P 2350 1300
-F 0 "D6" H 2300 1380 50  0000 L CNN
-F 1 "3V" H 2200 1250 50  0000 L CNN
-F 2 "Diodes_SMD:SOD-323" V 2350 1300 50  0001 C CNN
-F 3 "" V 2350 1300 50  0000 C CNN
-	1    2350 1300
-	0    1    1    0
-$EndComp
-$Comp
-L D_Schottky_Small D7
-U 1 1 57A22D00
-P 2450 1300
-F 0 "D7" H 2400 1380 50  0000 L CNN
-F 1 "3V" H 2300 1250 50  0000 L CNN
-F 2 "Diodes_SMD:SOD-323" V 2450 1300 50  0001 C CNN
-F 3 "" V 2450 1300 50  0000 C CNN
-	1    2450 1300
-	0    1    1    0
-$EndComp
-$Comp
-L D_Schottky_Small D9
-U 1 1 57A22D28
-P 2550 1300
-F 0 "D9" H 2500 1380 50  0000 L CNN
-F 1 "3V" H 2400 1250 50  0000 L CNN
-F 2 "Diodes_SMD:SOD-323" V 2550 1300 50  0001 C CNN
-F 3 "" V 2550 1300 50  0000 C CNN
-	1    2550 1300
-	0    1    1    0
-$EndComp
-Wire Wire Line
-	2400 1600 2400 1500
-Connection ~ 2400 1500
 $EndSCHEMATC

Commit message: updated stuff
Parts:
- RP3: value 1k -> 10k
Changed lines of the file:
@@
 $Descr A4 11693 8268
 encoding utf-8
-Sheet 7 13
+Sheet 6 12
 Title ""
 Date ""
@@
 P 1950 700
 F 0 "RP3" H 1950 1150 50  0000 C CNN
-F 1 "1k" H 1950 650 50  0000 C CNN
+F 1 "10k" H 1950 650 50  0000 C CNN
 F 2 "Resistors_SMD:R_Array_Concave_4x0603" H 1950 700 50  0001 C CNN
 F 3 "" H 1950 700 50  0000 C CNN

Commit message: i think im good with the schematics
Parts:
- added D? (x3): D_Schottky, symbol D_Schottky
- RP1: value 10k -> 20k
Connections:
- net GND: now also D?.2 (A), D?.2 (A), D?.2 (A)
- net OUT_1: now also D?.1 (K)
- net OUT_2: now also D?.1 (K)
- net OUT_3: now also D?.1 (K)
- net IN_4: no longer names the net of RP1.4 (P4)
- net OUT_4: no longer names the net of RP3.1 (P1)
- now unconnected: RP1.5 (R4), RP2.1 (P1), RP3.8 (R1)
Changed lines of the file:
@@
 Text HLabel 850  950  0    60   Input ~ 0
 IN_3
-Text HLabel 850  1050 0    60   Input ~ 0
-IN_4
 Wire Wire Line
 	950  750  850  750
@@
 Wire Wire Line
 	950  950  850  950
-Wire Wire Line
-	850  1050 950  1050
 $Comp
 L R_PACK4 RP1
@@
 P 1150 1100
 F 0 "RP1" H 1150 1550 50  0000 C CNN
-F 1 "10k" H 1150 1050 50  0000 C CNN
+F 1 "20k" H 1150 1050 50  0000 C CNN
 F 2 "Resistors_SMD:R_Array_Concave_4x0603" H 1150 1100 50  0001 C CNN
 F 3 "" H 1150 1100 50  0000 C CNN
@@
 $EndComp
 Wire Wire Line
-	1350 1050 1750 1050
-Wire Wire Line
 	1350 950  1750 950
 Wire Wire Line
@@
 	1600 1150 1600 950
 Connection ~ 1600 950
-Wire Wire Line
-	1700 1150 1700 1050
-Connection ~ 1700 1050
 Wire Wire Line
 	1400 1550 1400 1600
@@
 Connection ~ 1550 1600
 Wire Wire Line
-	2150 1050 2800 1050
-Wire Wire Line
 	2150 950  2800 950
 Wire Wire Line
@@
 Text HLabel 2800 950  2    60   Output ~ 0
 OUT_3
-Text HLabel 2800 1050 2    60   Output ~ 0
-OUT_4
+$Comp
+L D_Schottky D?
+U 1 1 580E2C17
+P 2250 1350
+F 0 "D?" H 2250 1450 50  0000 C CNN
+F 1 "D_Schottky" H 2250 1250 50  0000 C CNN
+F 2 "" H 2250 1350 50  0000 C CNN
+F 3 "" H 2250 1350 50  0000 C CNN
+	1    2250 1350
+	0    1    1    0
+$EndComp
+$Comp
+L D_Schottky D?
+U 1 1 580E2C46
+P 2400 1350
+F 0 "D?" H 2400 1450 50  0000 C CNN
+F 1 "D_Schottky" H 2400 1250 50  0000 C CNN
+F 2 "" H 2400 1350 50  0000 C CNN
+F 3 "" H 2400 1350 50  0000 C CNN
+	1    2400 1350
+	0    1    1    0
+$EndComp
+$Comp
+L D_Schottky D?
+U 1 1 580E2C67
+P 2550 1350
+F 0 "D?" H 2550 1450 50  0000 C CNN
+F 1 "D_Schottky" H 2550 1250 50  0000 C CNN
+F 2 "" H 2550 1350 50  0000 C CNN
+F 3 "" H 2550 1350 50  0000 C CNN
+	1    2550 1350
+	0    1    1    0
+$EndComp
+$Comp
+L GND #PWR?
+U 1 1 580E2CFB
+P 2400 1700
+F 0 "#PWR?" H 2400 1450 50  0001 C CNN
+F 1 "GND" H 2400 1550 50  0000 C CNN
+F 2 "" H 2400 1700 50  0000 C CNN
+F 3 "" H 2400 1700 50  0000 C CNN
+	1    2400 1700
+	1    0    0    -1
+$EndComp
+Wire Wire Line
+	2250 1650 2550 1650
+Wire Wire Line
+	2550 1650 2550 1500
+Wire Wire Line
+	2250 1650 2250 1500
+Wire Wire Line
+	2400 1500 2400 1700
+Connection ~ 2400 1650
+Wire Wire Line
+	2250 1200 2250 950
+Connection ~ 2250 950
+Wire Wire Line
+	2400 1200 2400 850
+Connection ~ 2400 850
+Wire Wire Line
+	2550 1200 2550 750
+Connection ~ 2550 750
 $EndSCHEMATC

Commit message: routed... at least for now
Parts:
- removed D? (x3): D_Schottky, symbol D_Schottky
- added D1, D2, D6, D7: 3.3V, Diodes_SMD:SOD-323, symbol ZENERsmall
Connections:
- net GND: now also D1.2 (A), D2.2 (A), D6.2 (A), D7.2 (A)
- net OUT_1: now also D6.1 (K)
- net OUT_2: now also D2.1 (K)
- net OUT_3: now also D1.1 (K)
- net IN_4: now reaches RP1.4 (P4)
- net at RP1.5 (R4): now also RP2.1 (P1), RP3.8 (R1)
- net OUT_4: now reaches RP3.1 (P1)
- net OUT_4: now also D7.1 (K)
Changed lines of the file:
@@
 Connection ~ 1500 1600
 $Comp
-L GND #PWR039
+L GND #PWR033
 U 1 1 57A226A1
 P 1550 1650
-F 0 "#PWR039" H 1550 1400 50  0001 C CNN
+F 0 "#PWR033" H 1550 1400 50  0001 C CNN
 F 1 "GND" H 1550 1500 50  0000 C CNN
 F 2 "" H 1550 1650 50  0000 C CNN
@@
 OUT_3
 $Comp
-L D_Schottky D?
-U 1 1 580E2C17
-P 2250 1350
-F 0 "D?" H 2250 1450 50  0000 C CNN
-F 1 "D_Schottky" H 2250 1250 50  0000 C CNN
-F 2 "" H 2250 1350 50  0000 C CNN
-F 3 "" H 2250 1350 50  0000 C CNN
-	1    2250 1350
+L GND #PWR034
+U 1 1 580E2CFB
+P 2500 1700
+F 0 "#PWR034" H 2500 1450 50  0001 C CNN
+F 1 "GND" H 2500 1550 50  0000 C CNN
+F 2 "" H 2500 1700 50  0000 C CNN
+F 3 "" H 2500 1700 50  0000 C CNN
+	1    2500 1700
+	1    0    0    -1
+$EndComp
+Wire Wire Line
+	2200 1650 2650 1650
+Wire Wire Line
+	2650 1650 2650 1450
+Wire Wire Line
+	2350 1650 2350 1450
+Wire Wire Line
+	2500 1450 2500 1700
+Connection ~ 2500 1650
+Wire Wire Line
+	2350 950  2350 1250
+Connection ~ 2350 950
+Wire Wire Line
+	2500 850  2500 1250
+Connection ~ 2500 850
+Wire Wire Line
+	2650 750  2650 1250
+Connection ~ 2650 750
+$Comp
+L ZENERsmall D1
+U 1 1 58135B64
+P 2350 1350
+F 0 "D1" H 2350 1450 50  0000 C CNN
+F 1 "3.3V" H 2350 1250 50  0000 C CNN
+F 2 "Diodes_SMD:SOD-323" H 2350 1350 50  0001 C CNN
+F 3 "" H 2350 1350 50  0000 C CNN
+	1    2350 1350
 	0    1    1    0
 $EndComp
 $Comp
-L D_Schottky D?
-U 1 1 580E2C46
-P 2400 1350
-F 0 "D?" H 2400 1450 50  0000 C CNN
-F 1 "D_Schottky" H 2400 1250 50  0000 C CNN
-F 2 "" H 2400 1350 50  0000 C CNN
-F 3 "" H 2400 1350 50  0000 C CNN
-	1    2400 1350
+L ZENERsmall D2
+U 1 1 58135C26
+P 2500 1350
+F 0 "D2" H 2500 1450 50  0000 C CNN
+F 1 "3.3V" H 2500 1250 50  0000 C CNN
+F 2 "Diodes_SMD:SOD-323" H 2500 1350 50  0001 C CNN
+F 3 "" H 2500 1350 50  0000 C CNN
+	1    2500 1350
 	0    1    1    0
 $EndComp
 $Comp
-L D_Schottky D?
-U 1 1 580E2C67
-P 2550 1350
-F 0 "D?" H 2550 1450 50  0000 C CNN
-F 1 "D_Schottky" H 2550 1250 50  0000 C CNN
-F 2 "" H 2550 1350 50  0000 C CNN
-F 3 "" H 2550 1350 50  0000 C CNN
-	1    2550 1350
+L ZENERsmall D6
+U 1 1 58135C47
+P 2650 1350
+F 0 "D6" H 2650 1450 50  0000 C CNN
+F 1 "3.3V" H 2650 1250 50  0000 C CNN
+F 2 "Diodes_SMD:SOD-323" H 2650 1350 50  0001 C CNN
+F 3 "" H 2650 1350 50  0000 C CNN
+	1    2650 1350
 	0    1    1    0
 $EndComp
+Text HLabel 850  1050 0    60   Input ~ 0
+IN_4
+Wire Wire Line
+	850  1050 950  1050
+Wire Wire Line
+	1350 1050 1750 1050
+Wire Wire Line
+	1700 1150 1700 1050
+Connection ~ 1700 1050
+Text HLabel 2800 1050 2    60   Output ~ 0
+OUT_4
+Wire Wire Line
+	2800 1050 2150 1050
 $Comp
-L GND #PWR?
-U 1 1 580E2CFB
-P 2400 1700
-F 0 "#PWR?" H 2400 1450 50  0001 C CNN
-F 1 "GND" H 2400 1550 50  0000 C CNN
-F 2 "" H 2400 1700 50  0000 C CNN
-F 3 "" H 2400 1700 50  0000 C CNN
-	1    2400 1700
-	1    0    0    -1
+L ZENERsmall D7
+U 1 1 5817BCDE
+P 2200 1350
+F 0 "D7" H 2200 1450 50  0000 C CNN
+F 1 "3.3V" H 2200 1250 50  0000 C CNN
+F 2 "Diodes_SMD:SOD-323" H 2200 1350 50  0001 C CNN
+F 3 "" H 2200 1350 50  0000 C CNN
+	1    2200 1350
+	0    1    1    0
 $EndComp
 Wire Wire Line
-	2250 1650 2550 1650
+	2200 1250 2200 1050
+Connection ~ 2200 1050
 Wire Wire Line
-	2550 1650 2550 1500
-Wire Wire Line
-	2250 1650 2250 1500
-Wire Wire Line
-	2400 1500 2400 1700
-Connection ~ 2400 1650
-Wire Wire Line
-	2250 1200 2250 950
-Connection ~ 2250 950
-Wire Wire Line
-	2400 1200 2400 850
-Connection ~ 2400 850
-Wire Wire Line
-	2550 1200 2550 750
-Connection ~ 2550 750
+	2200 1450 2200 1650
+Connection ~ 2350 1650
 $EndSCHEMATC

Commit message: long forgotten commit of something I did half a year ago -.-
Parts:
- removed D1, D2, D6, D7: 3.3V, Diodes_SMD:SOD-323, symbol ZENERsmall
- removed RP3: 10k, Resistors_SMD:R_Array_Concave_4x0603, symbol R_PACK4
- RP1, RP2: footprint Resistors_SMD:R_Array_Concave_4x0603 -> Resistor_SMD:R_Array_Concave_4x0603; symbol R_PACK4 -> bldc-controller-rescue:R_PACK4
Connections:
- net OUT_1: now also RP1.8 (R1), RP2.1 (P1)
- net OUT_2: now also RP1.7 (R2), RP2.2 (P2)
- net OUT_3: now also RP1.6 (R3), RP2.3 (P3)
- net OUT_4: now also RP1.5 (R4), RP2.4 (P4)
Changed lines of the file:
@@
-EESchema Schematic File Version 2
-LIBS:bldc-controller-rescue
-LIBS:power
-LIBS:device
-LIBS:transistors
-LIBS:conn
-LIBS:linear
-LIBS:regul
-LIBS:74xx
-LIBS:cmos4000
-LIBS:adc-dac
-LIBS:memory
-LIBS:xilinx
-LIBS:microcontrollers
-LIBS:dsp
-LIBS:microchip
-LIBS:analog_switches
-LIBS:motorola
-LIBS:texas
-LIBS:intel
-LIBS:audio
-LIBS:interface
-LIBS:digital-audio
-LIBS:philips
-LIBS:display
-LIBS:cypress
-LIBS:siliconi
-LIBS:opto
-LIBS:atmel
-LIBS:contrib
-LIBS:valves
-LIBS:Power_Management
-LIBS:st-microelectronics
-LIBS:stm32
-LIBS:w_analog
-LIBS:mpu6000
+EESchema Schematic File Version 4
 LIBS:bldc-controller-cache
-EELAYER 25 0
+EELAYER 29 0
 EELAYER END
 $Descr A4 11693 8268
@@
 	950  950  850  950
 $Comp
-L R_PACK4 RP1
+L bldc-controller-rescue:R_PACK4 RP1
 U 1 1 57A2245B
 P 1150 1100
 F 0 "RP1" H 1150 1550 50  0000 C CNN
 F 1 "20k" H 1150 1050 50  0000 C CNN
-F 2 "Resistors_SMD:R_Array_Concave_4x0603" H 1150 1100 50  0001 C CNN
+F 2 "Resistor_SMD:R_Array_Concave_4x0603" H 1150 1100 50  0001 C CNN
 F 3 "" H 1150 1100 50  0000 C CNN
 	1    1150 1100
@@
 $EndComp
 $Comp
-L R_PACK4 RP2
+L bldc-controller-rescue:R_PACK4 RP2
 U 1 1 57A22518
-P 1350 1350
-F 0 "RP2" H 1350 1800 50  0000 C CNN
-F 1 "1k" H 1350 1300 50  0000 C CNN
-F 2 "Resistors_SMD:R_Array_Concave_4x0603" H 1350 1350 50  0001 C CNN
-F 3 "" H 1350 1350 50  0000 C CNN
-	1    1350 1350
-	0    1    1    0
-$EndComp
-$Comp
-L R_PACK4 RP3
-U 1 1 57A2257E
-P 1950 700
-F 0 "RP3" H 1950 1150 50  0000 C CNN
-F 1 "10k" H 1950 650 50  0000 C CNN
-F 2 "Resistors_SMD:R_Array_Concave_4x0603" H 1950 700 50  0001 C CNN
-F 3 "" H 1950 700 50  0000 C CNN
-	1    1950 700
-	-1   0    0    1
+P 1750 1350
+F 0 "RP2" H 1750 1800 50  0000 C CNN
+F 1 "1k" H 1750 1300 50  0000 C CNN
+F 2 "Resistor_SMD:R_Array_Concave_4x0603" H 1750 1350 50  0001 C CNN
+F 3 "" H 1750 1350 50  0000 C CNN
+	1    1750 1350
+	0    -1   1    0
 $EndComp
 Wire Wire Line
-	1350 950  1750 950
+	1350 950  1600 950
 Wire Wire Line
-	1350 850  1750 850
+	1350 850  1500 850
 Wire Wire Line
-	1350 750  1750 750
+	1350 750  1400 750
 Wire Wire Line
 	1400 1150 1400 750
@@
 	1400 1550 1400 1600
 Wire Wire Line
-	1400 1600 1700 1600
+	1400 1600 1500 1600
 Wire Wire Line
 	1700 1600 1700 1550
@@
 Connection ~ 1500 1600
 $Comp
-L GND #PWR033
+L bldc-controller-rescue:GND #PWR033
 U 1 1 57A226A1
 P 1550 1650
@@
 	1550 1650 1550 1600
 Connection ~ 1550 1600
-Wire Wire Line
-	2150 950  2800 950
-Wire Wire Line
-	2150 850  2800 850
-Wire Wire Line
-	2150 750  2800 750
 Text HLabel 2800 750  2    60   Output ~ 0
 OUT_1
@@
 Text HLabel 2800 950  2    60   Output ~ 0
 OUT_3
-$Comp
-L GND #PWR034
-U 1 1 580E2CFB
-P 2500 1700
-F 0 "#PWR034" H 2500 1450 50  0001 C CNN
-F 1 "GND" H 2500 1550 50  0000 C CNN
-F 2 "" H 2500 1700 50  0000 C CNN
-F 3 "" H 2500 1700 50  0000 C CNN
-	1    2500 1700
-	1    0    0    -1
-$EndComp
-Wire Wire Line
-	2200 1650 2650 1650
-Wire Wire Line
-	2650 1650 2650 1450
-Wire Wire Line
-	2350 1650 2350 1450
-Wire Wire Line
-	2500 1450 2500 1700
-Connection ~ 2500 1650
-Wire Wire Line
-	2350 950  2350 1250
-Connection ~ 2350 950
-Wire Wire Line
-	2500 850  2500 1250
-Connection ~ 2500 850
-Wire Wire Line
-	2650 750  2650 1250
-Connection ~ 2650 750
-$Comp
-L ZENERsmall D1
-U 1 1 58135B64
-P 2350 1350
-F 0 "D1" H 2350 1450 50  0000 C CNN
-F 1 "3.3V" H 2350 1250 50  0000 C CNN
-F 2 "Diodes_SMD:SOD-323" H 2350 1350 50  0001 C CNN
-F 3 "" H 2350 1350 50  0000 C CNN
-	1    2350 1350
-	0    1    1    0
-$EndComp
-$Comp
-L ZENERsmall D2
-U 1 1 58135C26
-P 2500 1350
-F 0 "D2" H 2500 1450 50  0000 C CNN
-F 1 "3.3V" H 2500 1250 50  0000 C CNN
-F 2 "Diodes_SMD:SOD-323" H 2500 1350 50  0001 C CNN
-F 3 "" H 2500 1350 50  0000 C CNN
-	1    2500 1350
-	0    1    1    0
-$EndComp
-$Comp
-L ZENERsmall D6
-U 1 1 58135C47
-P 2650 1350
-F 0 "D6" H 2650 1450 50  0000 C CNN
-F 1 "3.3V" H 2650 1250 50  0000 C CNN
-F 2 "Diodes_SMD:SOD-323" H 2650 1350 50  0001 C CNN
-F 3 "" H 2650 1350 50  0000 C CNN
-	1    2650 1350
-	0    1    1    0
-$EndComp
 Text HLabel 850  1050 0    60   Input ~ 0
 IN_4
@@
 	850  1050 950  1050
 Wire Wire Line
-	1350 1050 1750 1050
+	1350 1050 1700 1050
 Wire Wire Line
 	1700 1150 1700 1050
@@
 OUT_4
 Wire Wire Line
-	2800 1050 2150 1050
-$Comp
-L ZENERsmall D7
-U 1 1 5817BCDE
-P 2200 1350
-F 0 "D7" H 2200 1450 50  0000 C CNN
-F 1 "3.3V" H 2200 1250 50  0000 C CNN
-F 2 "Diodes_SMD:SOD-323" H 2200 1350 50  0001 C CNN
-F 3 "" H 2200 1350 50  0000 C CNN
-	1    2200 1350
-	0    1    1    0
-$EndComp
+	1600 1600 1700 1600
 Wire Wire Line
-	2200 1250 2200 1050
-Connection ~ 2200 1050
+	1500 1600 1550 1600
 Wire Wire Line
-	2200 1450 2200 1650
-Connection ~ 2350 1650
+	1550 1600 1600 1600
+Wire Wire Line
+	1400 750  2800 750
+Wire Wire Line
+	1500 850  2800 850
+Wire Wire Line
+	1600 950  2800 950
+Wire Wire Line
+	1700 1050 2800 1050
 $EndSCHEMATC
