File: Holes.sch (KiCad schematic (older format))
At the start: 0 parts

Commit message: fertig?
Parts:
- added P10, P2, P8, P9: MOUNTING, Connect:1pin, symbol CONN_01X01
Connections:
- no-connect marks 0 -> 4
Changed lines of the file:
@@
 $Descr A4 11693 8268
 encoding utf-8
-Sheet 13 12
+Sheet 12 13
 Title ""
 Date ""
@@
 Comment4 ""
 $EndDescr
+$Comp
+L CONN_01X01 P2
+U 1 1 57B69B90
+P 850 700
+F 0 "P2" H 850 800 50  0000 C CNN
+F 1 "MOUNTING" V 950 700 50  0000 C CNN
+F 2 "Connect:1pin" H 850 700 50  0001 C CNN
+F 3 "" H 850 700 50  0000 C CNN
+	1    850  700
+	1    0    0    -1
+$EndComp
+$Comp
+L CONN_01X01 P9
+U 1 1 57B69C12
+P 1200 700
+F 0 "P9" H 1200 800 50  0000 C CNN
+F 1 "MOUNTING" V 1300 700 50  0000 C CNN
+F 2 "Connect:1pin" H 1200 700 50  0001 C CNN
+F 3 "" H 1200 700 50  0000 C CNN
+	1    1200 700
+	1    0    0    -1
+$EndComp
+$Comp
+L CONN_01X01 P8
+U 1 1 57B69C4E
+P 850 1100
+F 0 "P8" H 850 1200 50  0000 C CNN
+F 1 "MOUNTING" V 950 1100 50  0000 C CNN
+F 2 "Connect:1pin" H 850 1100 50  0001 C CNN
+F 3 "" H 850 1100 50  0000 C CNN
+	1    850  1100
+	1    0    0    -1
+$EndComp
+$Comp
+L CONN_01X01 P10
+U 1 1 57B69C7B
+P 1200 1100
+F 0 "P10" H 1200 1200 50  0000 C CNN
+F 1 "MOUNTING" V 1300 1100 50  0000 C CNN
+F 2 "Connect:1pin" H 1200 1100 50  0001 C CNN
+F 3 "" H 1200 1100 50  0000 C CNN
+	1    1200 1100
+	1    0    0    -1
+$EndComp
+NoConn ~ 650  700
+NoConn ~ 1000 700
+NoConn ~ 1000 1100
+NoConn ~ 650  1100
 $EndSCHEMATC

Commit message: long forgotten commit of something I did half a year ago -.-
Parts:
- P10, P2, P8, P9: symbol CONN_01X01 -> bldc-controller-rescue:CONN_01X01
Changed lines of the file:
@@
-EESchema Schematic File Version 2
-LIBS:bldc-controller-rescue
-LIBS:power
-LIBS:device
-LIBS:transistors
-LIBS:conn
-LIBS:linear
-LIBS:regul
-LIBS:74xx
-LIBS:cmos4000
-LIBS:adc-dac
-LIBS:memory
-LIBS:xilinx
-LIBS:microcontrollers
-LIBS:dsp
-LIBS:microchip
-LIBS:analog_switches
-LIBS:motorola
-LIBS:texas
-LIBS:intel
-LIBS:audio
-LIBS:interface
-LIBS:digital-audio
-LIBS:philips
-LIBS:display
-LIBS:cypress
-LIBS:siliconi
-LIBS:opto
-LIBS:atmel
-LIBS:contrib
-LIBS:valves
-LIBS:Power_Management
-LIBS:st-microelectronics
-LIBS:stm32
-LIBS:w_analog
-LIBS:mpu6000
+EESchema Schematic File Version 4
 LIBS:bldc-controller-cache
-EELAYER 25 0
+EELAYER 29 0
 EELAYER END
 $Descr A4 11693 8268
 encoding utf-8
-Sheet 12 12
+Sheet 9 12
 Title ""
 Date ""
@@
 $EndDescr
 $Comp
-L CONN_01X01 P2
+L bldc-controller-rescue:CONN_01X01 P2
 U 1 1 57B69B90
 P 850 700
@@
 $EndComp
 $Comp
-L CONN_01X01 P9
+L bldc-controller-rescue:CONN_01X01 P9
 U 1 1 57B69C12
 P 1200 700
@@
 $EndComp
 $Comp
-L CONN_01X01 P8
+L bldc-controller-rescue:CONN_01X01 P8
 U 1 1 57B69C4E
 P 850 1100
@@
 $EndComp
 $Comp
-L CONN_01X01 P10
+L bldc-controller-rescue:CONN_01X01 P10
 U 1 1 57B69C7B
 P 1200 1100
