File: SWDIO.sch (KiCad schematic (older format))
At the start: 1 part, among them P5 CONN_01X05

Commit message: blubb
Parts:
- P5: value CONN_01X05 -> CON_SWD; footprint Pin_Headers:Pin_Header_Angled_1x05 -> Socket_Strips:Socket_Strip_Straight_1x05
Changed lines of the file:
@@
 EESchema Schematic File Version 2
+LIBS:bldc-controller-rescue
 LIBS:power
 LIBS:device
@@
 LIBS:st-microelectronics
 LIBS:stm32
+LIBS:w_analog
+LIBS:mpu6000
 LIBS:bldc-controller-cache
 EELAYER 25 0
@@
 $Descr A4 11693 8268
 encoding utf-8
-Sheet 6 6
+Sheet 6 13
 Title "DreErolf"
 Date ""
@@
 	1200 4800 1500 4800
 $Comp
-L GND #PWR046
+L GND #PWR025
 U 1 1 577BF039
 P 1200 4900
-F 0 "#PWR046" H 1200 4650 50  0001 C CNN
+F 0 "#PWR025" H 1200 4650 50  0001 C CNN
 F 1 "GND" H 1200 4750 50  0000 C CNN
 F 2 "" H 1200 4900 50  0000 C CNN
@@
 	1200 4400 1500 4400
 $Comp
-L VCC #PWR047
+L VCC #PWR026
 U 1 1 577BF056
 P 1200 4300
-F 0 "#PWR047" H 1200 4150 50  0001 C CNN
+F 0 "#PWR026" H 1200 4150 50  0001 C CNN
 F 1 "VCC" H 1200 4450 50  0000 C CNN
 F 2 "" H 1200 4300 50  0000 C CNN
@@
 P 1700 4600
 F 0 "P5" H 1700 4900 50  0000 C CNN
-F 1 "CONN_01X05" V 1800 4600 50  0000 C CNN
-F 2 "Pin_Headers:Pin_Header_Angled_1x05" H 1700 4600 50  0001 C CNN
+F 1 "CON_SWD" V 1800 4600 50  0000 C CNN
+F 2 "Socket_Strips:Socket_Strip_Straight_1x05" H 1700 4600 50  0001 C CNN
 F 3 "" H 1700 4600 50  0000 C CNN
 	1    1700 4600

Commit message: long forgotten commit of something I did half a year ago -.-
Parts:
- P5: footprint Socket_Strips:Socket_Strip_Straight_1x05 -> Connector_PinHeader_2.54mm:PinHeader_1x05_P2.54mm_Vertical; symbol CONN_01X05 -> bldc-controller-rescue:CONN_01X05
Changed lines of the file:
@@
-EESchema Schematic File Version 2
-LIBS:bldc-controller-rescue
-LIBS:power
-LIBS:device
-LIBS:transistors
-LIBS:conn
-LIBS:linear
-LIBS:regul
-LIBS:74xx
-LIBS:cmos4000
-LIBS:adc-dac
-LIBS:memory
-LIBS:xilinx
-LIBS:microcontrollers
-LIBS:dsp
-LIBS:microchip
-LIBS:analog_switches
-LIBS:motorola
-LIBS:texas
-LIBS:intel
-LIBS:audio
-LIBS:interface
-LIBS:digital-audio
-LIBS:philips
-LIBS:display
-LIBS:cypress
-LIBS:siliconi
-LIBS:opto
-LIBS:atmel
-LIBS:contrib
-LIBS:valves
-LIBS:Power_Management
-LIBS:st-microelectronics
-LIBS:stm32
-LIBS:w_analog
-LIBS:mpu6000
+EESchema Schematic File Version 4
 LIBS:bldc-controller-cache
-EELAYER 25 0
+EELAYER 29 0
 EELAYER END
 $Descr A4 11693 8268
@@
 	1200 4800 1500 4800
 $Comp
-L GND #PWR019
+L bldc-controller-rescue:GND #PWR019
 U 1 1 577BF039
 P 1200 4900
@@
 	1200 4400 1500 4400
 $Comp
-L VCC #PWR020
+L bldc-controller-rescue:VCC #PWR020
 U 1 1 577BF056
 P 1200 4300
+AR Path="/577BF056" Ref="#PWR020"  Part="1"
+AR Path="/578EBA53/577BF056" Ref="#PWR020"  Part="1"
 F 0 "#PWR020" H 1200 4150 50  0001 C CNN
 F 1 "VCC" H 1200 4450 50  0000 C CNN
@@
 	1200 4400 1200 4300
 $Comp
-L CONN_01X05 P5
+L bldc-controller-rescue:CONN_01X05 P5
 U 1 1 577BF0D1
 P 1700 4600
 F 0 "P5" H 1700 4900 50  0000 C CNN
 F 1 "CON_SWD" V 1800 4600 50  0000 C CNN
-F 2 "Socket_Strips:Socket_Strip_Straight_1x05" H 1700 4600 50  0001 C CNN
+F 2 "Connector_PinHeader_2.54mm:PinHeader_1x05_P2.54mm_Vertical" H 1700 4600 50  0001 C CNN
 F 3 "" H 1700 4600 50  0000 C CNN
 	1    1700 4600
